Commit message: Add raspicam to urdf, remove static transform

File: magni_description/urdf/basic_magni.urdf (robot description, URDF)
Before this commit: robot magni, 3 links, 2 joints
Links:
- added link raspicam
Joints:
- added joint raspicam_joint: type fixed, parent base_link, child raspicam, origin xyz=0.035 0.145 0.14 rpy=0 -1.5707 0

Commit message: Fix camera transform

File: magni_description/urdf/basic_magni.urdf (robot description, URDF)
Before this commit: robot magni, 4 links, 3 joints
Joints:
- joint raspicam_joint: origin xyz=0.035 0.145 0.14 rpy=0 -1.5707 0 -> xyz=0.035 0.145 0.14 rpy=0 0 0

Commit message: swap left and right wheel positions, fixes #22

File: magni_description/urdf/basic_magni.urdf (robot description, URDF)
Before this commit: robot magni, 4 links, 3 joints
Joints:
- joint left_wheel_joint: origin xyz=0 -0.165 -0.057704 rpy=0 0 0 -> xyz=0 0.165 -0.057704 rpy=0 0 0
- joint right_wheel_joint: origin xyz=0 0.165 -0.057704 rpy=3.14 0 0 -> xyz=0 -0.165 -0.057704 rpy=3.14 0 0

Commit message: Rotated the camera 180 degrees

File: magni_description/urdf/basic_magni.urdf (robot description, URDF)
Before this commit: robot magni, 4 links, 3 joints
Joints:
- joint raspicam_joint: origin xyz=0.035 0.145 0.14 rpy=0 0 0 -> xyz=0.035 0.145 0.14 rpy=0 0 3.1416
