Commit message: Gazebo integration updates.

File: magni_description/urdf/inertial.xacro (robot description, xacro)
@@ -1,8 +1,28 @@
 <?xml version="1.0"?>
 <!--
-Copyright: Osnabrück University, Knowledge Based Systems Group
-https://raw.githubusercontent.com/uos/uos_tools/kinetic/uos_common_urdf/common.xacro
+Copyright 2019 Osnabrück University, Knowledge Based Systems Group
+https://github.com/uos/uos_tools/tree/kinetic/uos_common_urdf
+Redistribution and use in source and binary forms, with or without modification,
+are permitted provided that the following conditions are met:
+1. Redistributions of source code must retain the above copyright notice,
+   this list of conditions and the following disclaimer.
+2. Redistributions in binary form must reproduce the above copyright notice,
+   this list of conditions and the following disclaimer in the documentation
+   and/or other materials provided with the distribution.
+3. Neither the name of the copyright holder nor the names of its contributors
+   may be used to endorse or promote products derived from this software without
+   specific prior written permission.
+THIS SOFTWARE IS PROVIDED BY THE COPYRIGHT HOLDERS AND CONTRIBUTORS "AS IS"
+AND ANY EXPRESS OR IMPLIED WARRANTIES, INCLUDING, BUT NOT LIMITED TO, THE IMPLIED
+WARRANTIES OF MERCHANTABILITY AND FITNESS FOR A PARTICULAR PURPOSE ARE DISCLAIMED.
+IN NO EVENT SHALL THE COPYRIGHT HOLDER OR CONTRIBUTORS BE LIABLE FOR ANY DIRECT,
+INDIRECT, INCIDENTAL, SPECIAL, EXEMPLARY, OR CONSEQUENTIAL DAMAGES (INCLUDING,
+BUT NOT LIMITED TO, PROCUREMENT OF SUBSTITUTE GOODS OR SERVICES; LOSS OF USE, DATA,
+OR PROFITS; OR BUSINESS INTERRUPTION) HOWEVER CAUSED AND ON ANY THEORY OF LIABILITY,
+WHETHER IN CONTRACT, STRICT LIABILITY, OR TORT (INCLUDING NEGLIGENCE OR OTHERWISE)
+ARISING IN ANY WAY OUT OF THE USE OF THIS SOFTWARE, EVEN IF ADVISED OF THE POSSIBILITY
+OF SUCH DAMAGE.
 -->
-<robot xmlns:xacro="http://ros.org/wiki/xacro">
+<robot xmlns:xacro="http://wiki.ros.org/xacro">
     <property name="M_PI" value="3.1415926535897931" />
     <!-- see https://secure.wikimedia.org/wikipedia/en/wiki/List_of_moment_of_inertia_tensors -->

File: magni_description/urdf/magni.urdf.xacro (robot description, xacro)
@@ -81,5 +81,5 @@
       </collision>
       <collision>
-        <origin xyz="0.033 0 0" rpy="0 ${pi/2} 0" />
+        <origin xyz="${0.033*reflect} 0 0" rpy="0 ${pi/2} 0" />
         <geometry>
           <cylinder radius="0.064" length="0.016"/>

Commit message: fixed magni tipping over

File: magni_description/urdf/inertial.xacro (robot description, xacro)
@@ -49,5 +49,5 @@
         <inertial>
             <mass value="${mass}" />
-            <origin xyz="0 0 0" />
+            <origin xyz="-0.15 0 0.03" />
             <inertia ixx="${0.0833333 * mass * (y*y + z*z)}" ixy="0.0" ixz="0.0"
                      iyy="${0.0833333 * mass * (x*x + z*z)}" iyz="0.0"
@@ -59,5 +59,5 @@
         <inertial>
             <mass value="${mass}" />
-            <insert_block name="origin" />
+            <xacro:insert_block name="origin" />
             <inertia ixx="${0.4 * mass * radius * radius}" ixy="0.0" ixz="0.0"
                      iyy="${0.4 * mass * radius * radius}" iyz="0.0"
@@ -68,5 +68,5 @@
         <inertial>
             <mass value="${mass}" />
-            <insert_block name="origin" />
+            <xacro:insert_block name="origin" />
             <inertia ixx="${0.0833333 * mass * (3 * radius * radius + length * length)}" ixy="0.0" ixz="0.0"
                      iyy="${0.0833333 * mass * (3 * radius * radius + length * length)}" iyz="0.0"
@@ -77,5 +77,5 @@
         <inertial>
             <mass value="${mass}" />
-            <insert_block name="origin" />
+            <xacro:insert_block name="origin" />
             <inertia ixx="${0.0833333 * mass * (y*y + z*z)}" ixy="0.0" ixz="0.0"
                      iyy="${0.0833333 * mass * (x*x + z*z)}" iyz="0.0"

Commit message: "Deprecated: xacro tag..." warning fixed

File: magni_description/urdf/inertial.xacro (robot description, xacro)
@@ -25,5 +25,5 @@
 -->
 <robot xmlns:xacro="http://wiki.ros.org/xacro">
-    <property name="M_PI" value="3.1415926535897931" />
+    <xacro:property name="M_PI" value="3.1415926535897931" />
     <!-- see https://secure.wikimedia.org/wikipedia/en/wiki/List_of_moment_of_inertia_tensors -->
     <!-- #################### versions without origin #################### -->

File: magni_gazebo/urdf/fiducials/aruco_marker.xacro (robot description, xacro)
@@ -5,5 +5,5 @@
                 <parent link="world"/>
                 <child link="${prefix}${marker_id}base_link"/>
-                <insert_block name="origin"/>
+                <xacro:insert_block name="origin"/>
             </joint>
         </xacro:if>
