Commit message: Robot mesh files added. Robot geometry description added to the URDF file.

File: magni_description/urdf/magni.urdf.xacro (robot description, xacro)
@@ -5,31 +5,110 @@
   <xacro:arg name="sonars_installed" default="true"/>
   <xacro:property name="sonars_installed" value="$(arg sonars_installed)"/>
-  <!-- base links for the urdf -->
-  <link name="base_link"/>
+  <xacro:property name="wheel_r" value="0.1" />
+  <xacro:property name="wheel_xpos" value="0.11" />
+  <!-- Inertia macro -->
+  <xacro:macro name="default_inertial" params="mass">
+    <inertial>
+      <mass value="${mass}" />
+      <inertia ixx="1.0" ixy="0.0" ixz="0.0" iyy="1.0" iyz="0.0" izz="1.0" />
+    </inertial>
+  </xacro:macro>
+  <!-- Robot base_link -->
+  <link name="base_link">
+    <visual>
+      <origin xyz="${-wheel_xpos} 0 ${-wheel_r+0.071}" rpy="0 0 0" />
+      <geometry>
+        <mesh filename="package://magni_description/meshes/magni_body.dae" />
+      </geometry>
+    </visual>
+	<visual>
+      <origin xyz="${-wheel_xpos-0.169} 0.17 ${-wheel_r+0.09}" rpy="0 0 ${pi}" />
+      <geometry>
+        <mesh filename="package://magni_description/meshes/caster_wheel.dae" />
+      </geometry>
+    </visual>
+	<visual>
+      <origin xyz="${-wheel_xpos-0.169} -0.17 ${-wheel_r+0.09}" rpy="0 0 ${pi}" />
+      <geometry>
+        <mesh filename="package://magni_description/meshes/caster_wheel.dae" />
+      </geometry>
+    </visual>
+    <collision>
+	  <origin xyz="${-wheel_xpos} 0 ${-wheel_r+0.151}" rpy="0 0 0" />
+      <geometry>
+        <box size="0.398 0.268 0.160"/>
+      </geometry>
+    </collision>
+    <collision>
+      <origin xyz="${-wheel_xpos-0.026} 0 ${-wheel_r+0.248}" rpy="0 0 0" />
+      <geometry>
+        <box size="0.375 0.268 0.034"/>
+      </geometry>
+    </collision>
+    <collision>
+      <origin xyz="${-wheel_xpos-0.169} 0.169 ${-wheel_r+0.106}" rpy="0 0 0" />
+      <geometry>
+        <box size="0.1 0.07 0.07"/>
+      </geometry>
+    </collision>
+    <collision>
+      <origin xyz="${-wheel_xpos-0.169} -0.169 ${-wheel_r+0.106}" rpy="0 0 0" />
+      <geometry>
+        <box size="0.1 0.07 0.07"/>
+      </geometry>
+    </collision>
+    <collision>
+      <origin xyz="${-wheel_xpos-0.19} 0.169 ${-wheel_r+0.04}" rpy="0 0 0" />
+      <geometry>
+        <sphere radius="0.04"/>
+      </geometry>
+    </collision>
+    <collision>
+      <origin xyz="${-wheel_xpos-0.19} -0.169 ${-wheel_r+0.04}" rpy="0 0 0" />
+      <geometry>
+        <sphere radius="0.04"/>
+      </geometry>
+    </collision>
+    <xacro:default_inertial mass="10"/>
+  </link>
+  <!-- Fixed offset from the floor to the center of the wheels -->
   <link name="base_footprint"/>
-  <!-- Fixed offset from the floor to the center of the wheels -->
   <joint name="base_footprint_joint" type="fixed">
     <parent link="base_link"/>
     <child link="base_footprint"/>
-    <origin xyz="0 0 -0.1" rpy="0 0 0"/>
+    <origin xyz="0 0 ${-wheel_r}" rpy="0 0 0"/>
   </joint>
   <!-- Macro for defining wheels -->
-  <xacro:macro name="wheel" params="name">
-    <link name="${name}_wheel"/>
-    <joint name="${name}_wheel_joint" type="continuous">
+  <xacro:macro name="wheel" params="prefix reflect">
+    <link name="${prefix}_wheel">
+      <visual>
+        <origin xyz="-0.071 0 0" rpy="0 0 0" />
+        <geometry>
+          <mesh filename="package://magni_description/meshes/front_wheel.dae" />
+        </geometry>
+      </visual>
+      <collision>
+        <origin xyz="0 0 0" rpy="0 ${pi/2} 0" />
+        <geometry>
+          <cylinder radius="${wheel_r}" length="0.05"/>
+        </geometry>
+      </collision>
+      <collision>
+        <origin xyz="0.033 0 0" rpy="0 ${pi/2} 0" />
+        <geometry>
+          <cylinder radius="0.064" length="0.016"/>
+        </geometry>
+      </collision>
+      <xacro:default_inertial mass="2"/>
+    </link>
+    <joint name="${prefix}_wheel_joint" type="continuous">
+      <axis xyz="0 1 0" rpy="0 0 0" />
       <parent link="base_link"/>
-      <child link="${name}_wheel"/>
-      <xacro:if value="${name == 'left'}">
-        <origin xyz="0 0.165 0" rpy="0 0 0" />
-        <axis xyz="0 1 0" />
-      </xacro:if>
-      <xacro:if value="${name == 'right'}">
-        <origin xyz="0 -0.165 0" rpy="${pi} 0 0" />
-        <axis xyz="0 -1 0" />
-      </xacro:if>
+      <child link="${prefix}_wheel"/>
+      <origin xyz="0 ${0.163*reflect} 0" rpy="0 0 ${pi/2 * reflect}"/>
     </joint>
   </xacro:macro>
-  <xacro:wheel name="left"/>
-  <xacro:wheel name="right"/>
+  <xacro:wheel prefix="left" reflect="1"/>
+  <xacro:wheel prefix="right" reflect="-1"/>
   <!-- Macro for defining sonars -->
   <xacro:macro name="sonar" params="name *origin">

Commit message: Fix wheel rotation axis

File: magni_description/urdf/magni.urdf.xacro (robot description, xacro)
@@ -103,5 +103,5 @@
     </link>
     <joint name="${prefix}_wheel_joint" type="continuous">
-      <axis xyz="0 1 0" rpy="0 0 0" />
+      <axis xyz="${1 * reflect } 0 0" rpy="0 0 0" />
       <parent link="base_link"/>
       <child link="${prefix}_wheel"/>

Commit message: Gazebo package added and URDF description update for Magni robot simulation

File: magni_description/urdf/magni.urdf.xacro (robot description, xacro)
@@ -1,4 +1,4 @@
 <?xml version="1.0"?>
-<robot xmlns:xacro="http://www.ros.org/wiki/xacro" name="magni">
+<robot xmlns:xacro="http://wiki.ros.org/xacro" name="magni">
   <xacro:arg name="raspicam_mount" default="forward"/>
   <xacro:property name="raspicam_mount" value="$(arg raspicam_mount)"/>
@@ -7,11 +7,7 @@
   <xacro:property name="wheel_r" value="0.1" />
   <xacro:property name="wheel_xpos" value="0.11" />
-  <!-- Inertia macro -->
-  <xacro:macro name="default_inertial" params="mass">
-    <inertial>
-      <mass value="${mass}" />
-      <inertia ixx="1.0" ixy="0.0" ixz="0.0" iyy="1.0" iyz="0.0" izz="1.0" />
-    </inertial>
-  </xacro:macro>
+  <xacro:include filename="$(find magni_description)/urdf/magni.transmission.xacro" />
+  <xacro:include filename="$(find magni_description)/urdf/magni.gazebo.xacro" />
+  <xacro:include filename="$(find magni_description)/urdf/inertial.xacro" />
   <!-- Robot base_link -->
   <link name="base_link">
@@ -58,24 +54,14 @@
       </geometry>
     </collision>
-    <collision>
-      <origin xyz="${-wheel_xpos-0.19} 0.169 ${-wheel_r+0.04}" rpy="0 0 0" />
-      <geometry>
-        <sphere radius="0.04"/>
-      </geometry>
-    </collision>
-    <collision>
-      <origin xyz="${-wheel_xpos-0.19} -0.169 ${-wheel_r+0.04}" rpy="0 0 0" />
-      <geometry>
-        <sphere radius="0.04"/>
-      </geometry>
-    </collision>
-    <xacro:default_inertial mass="10"/>
+    <xacro:box_inertial_with_origin  x="0.398" y="0.221" z="0.150" mass="10.0">
+      <origin xyz="-0.15 0 0.03" rpy="0 0 0" />
+    </xacro:box_inertial_with_origin>
   </link>
   <!-- Fixed offset from the floor to the center of the wheels -->
   <link name="base_footprint"/>
   <joint name="base_footprint_joint" type="fixed">
-    <parent link="base_link"/>
-    <child link="base_footprint"/>
-    <origin xyz="0 0 ${-wheel_r}" rpy="0 0 0"/>
+    <parent link="base_footprint"/>
+    <child link="base_link"/>
+    <origin xyz="0 0 ${wheel_r}" rpy="0 0 0"/>
   </joint>
   <!-- Macro for defining wheels -->
@@ -83,5 +69,5 @@
     <link name="${prefix}_wheel">
       <visual>
-        <origin xyz="-0.071 0 0" rpy="0 0 0" />
+        <origin xyz="${-0.071*reflect} 0 0" rpy="0 ${(reflect-1)*pi/2} 0" />
         <geometry>
           <mesh filename="package://magni_description/meshes/front_wheel.dae" />
@@ -100,15 +86,34 @@
         </geometry>
       </collision>
-      <xacro:default_inertial mass="2"/>
+      <xacro:cylinder_inertial_with_origin radius="${wheel_r}" length="0.05" mass="3.34">
+        <origin xyz="0 0 0" rpy="0 ${pi/2} 0" />
+      </xacro:cylinder_inertial_with_origin>
     </link>
     <joint name="${prefix}_wheel_joint" type="continuous">
-      <axis xyz="0 1 0" rpy="0 0 0" />
+      <axis xyz="1 0 0" rpy="0 0 0" />
       <parent link="base_link"/>
       <child link="${prefix}_wheel"/>
-      <origin xyz="0 ${0.163*reflect} 0" rpy="0 0 ${pi/2 * reflect}"/>
+      <origin xyz="0 ${0.163*reflect} 0" rpy="0 0 ${pi/2}"/>
     </joint>
   </xacro:macro>
   <xacro:wheel prefix="left" reflect="1"/>
   <xacro:wheel prefix="right" reflect="-1"/>
+  <!-- Macro for defining caster wheels -->
+  <xacro:macro name="caster_wheel" params="prefix reflect">
+    <link name="${prefix}_caster_wheel">
+      <collision>
+        <origin xyz="${-wheel_xpos-0.19} ${reflect*0.169} ${-wheel_r+0.04}" rpy="0 0 0" />
+        <geometry>
+          <sphere radius="0.04"/>
+        </geometry>
+      </collision>
+    </link>
+    <joint name="${prefix}_caster_wheel_joint" type="fixed">
+      <parent link="base_link"/>
+      <child link="${prefix}_caster_wheel"/>
+    </joint>
+  </xacro:macro>
+  <xacro:caster_wheel prefix="left" reflect="1"/>
+  <xacro:caster_wheel prefix="right" reflect="-1"/>
   <!-- Macro for defining sonars -->
   <xacro:macro name="sonar" params="name *origin">

Commit message: Sensors simulation in Gazebo added.

File: magni_description/urdf/magni.urdf.xacro (robot description, xacro)
@@ -10,4 +10,6 @@
   <xacro:include filename="$(find magni_description)/urdf/magni.gazebo.xacro" />
   <xacro:include filename="$(find magni_description)/urdf/inertial.xacro" />
+  <xacro:include filename="$(find magni_description)/urdf/sensors/sonar_hc-sr04.xacro" />
+  <xacro:include filename="$(find magni_description)/urdf/sensors/raspi_camera.xacro" />
   <!-- Robot base_link -->
   <link name="base_link">
@@ -116,50 +118,41 @@
   <xacro:caster_wheel prefix="left" reflect="1"/>
   <xacro:caster_wheel prefix="right" reflect="-1"/>
-  <!-- Macro for defining sonars -->
-  <xacro:macro name="sonar" params="name *origin">
-    <link name="${name}"/>
-    <joint name="${name}" type="fixed">
-      <parent link="base_link"/>
-      <child link="${name}"/>
-      <xacro:insert_block name="origin"/>
-    </joint>
-  </xacro:macro>
   <!-- Define all sonars, if sonars_installed set to 1 -->
   <xacro:if value="${sonars_installed}">
-    <xacro:sonar name="sonar_0">
+    <xacro:sonar_hc-sr04 name="sonar_0" connected_to="base_link">
       <origin xyz="0.01 -0.14 0.15" rpy="0 0 ${-pi/2}"/>
-    </xacro:sonar>
-    <xacro:sonar name="sonar_1">
+    </xacro:sonar_hc-sr04>
+    <xacro:sonar_hc-sr04 name="sonar_1" connected_to="base_link">
       <origin xyz="0.08 -0.07 0.15" rpy="0 0 0.785"/>
-    </xacro:sonar>
-    <xacro:sonar name="sonar_2">
+    </xacro:sonar_hc-sr04>
+    <xacro:sonar_hc-sr04 name="sonar_2" connected_to="base_link">
       <origin xyz="0.08 -0.01 0.15" rpy="0 0 -0.785"/>
-    </xacro:sonar>
-    <xacro:sonar name="sonar_3">
+    </xacro:sonar_hc-sr04>
+    <xacro:sonar_hc-sr04 name="sonar_3" connected_to="base_link">
       <origin xyz="0.08 0.04 0.15" rpy="0 0 0"/>
-    </xacro:sonar>
-    <xacro:sonar name="sonar_4">
+    </xacro:sonar_hc-sr04>
+    <xacro:sonar_hc-sr04 name="sonar_4" connected_to="base_link">
       <origin xyz="0.01 0.14 0.15" rpy="0 0 ${pi/2}"/>
-    </xacro:sonar>
+    </xacro:sonar_hc-sr04>
   </xacro:if>
-  <!-- Macro for defining raspicam -->
-  <xacro:macro name="raspicam" params="*origin">
-    <link name="raspicam"/>
-    <joint name="raspicam" type="fixed">
-      <parent link="base_link"/>
-      <child link="raspicam"/>
-      <xacro:insert_block name="origin"/>
-    </joint>
-  </xacro:macro>
+  <!--&lt;!&ndash; Macro for defining raspicam &ndash;&gt;-->
+  <!--<xacro:macro name="raspicam" params="*origin">-->
+    <!--<link name="raspicam"/>-->
+    <!--<joint name="raspicam" type="fixed">-->
+      <!--<parent link="base_link"/>-->
+      <!--<child link="raspicam"/>-->
+      <!--<xacro:insert_block name="origin"/>-->
+    <!--</joint>-->
+  <!--</xacro:macro>-->
   <!-- Define raspicam based on the raspicam_mount argument -->
   <xacro:if value="${raspicam_mount == 'forward'}">
-    <xacro:raspicam>
+    <xacro:raspi_camera name="raspicam" connected_to="base_link">
       <origin xyz="0.035 0.085 0.14" rpy="1.15191731 0 1.5707"/>
-    </xacro:raspicam>
+    </xacro:raspi_camera>
   </xacro:if>
   <xacro:if value="${raspicam_mount == 'upward'}">
-    <xacro:raspicam>
+    <xacro:raspi_camera name="raspicam" connected_to="base_link">
       <origin xyz="0.035 0.15 0.14" rpy="0 0 ${pi}"/>
-    </xacro:raspicam>
+    </xacro:raspi_camera>
   </xacro:if>
 </robot>

Commit message: Sensors corrections.

File: magni_description/urdf/magni.urdf.xacro (robot description, xacro)
@@ -136,13 +136,4 @@
     </xacro:sonar_hc-sr04>
   </xacro:if>
-  <!--&lt;!&ndash; Macro for defining raspicam &ndash;&gt;-->
-  <!--<xacro:macro name="raspicam" params="*origin">-->
-    <!--<link name="raspicam"/>-->
-    <!--<joint name="raspicam" type="fixed">-->
-      <!--<parent link="base_link"/>-->
-      <!--<child link="raspicam"/>-->
-      <!--<xacro:insert_block name="origin"/>-->
-    <!--</joint>-->
-  <!--</xacro:macro>-->
   <!-- Define raspicam based on the raspicam_mount argument -->
   <xacro:if value="${raspicam_mount == 'forward'}">

File: magni_description/urdf/sensors/raspi_camera.xacro (robot description, xacro)
@@ -17,7 +17,7 @@
       </visual>
       <collision>
-        <origin xyz="0.01 0 0" rpy="0 0 0" />
+        <origin xyz="0 0 0" rpy="0 0 ${pi/2}" />
         <geometry>
-          <box size="0.02 0.04 0.04"/>
+          <box size="0.03 0.026 0.016"/>
         </geometry>
       </collision>
@@ -28,13 +28,13 @@
       <parent link="${name}"/>
       <child link="${name}_sensor"/>
-      <origin xyz="0 0 0" rpy="${pi/2} ${-pi/2} 0" />
+      <origin xyz="0 0 0.012" rpy="${pi/2} ${-pi/2} 0" />
     </joint>
     <!-- Gazebo sensor plugin -->
     <gazebo reference="${name}_sensor">
       <sensor type="camera" name="camera1">
-        <visualize>false</visualize>
+        <visualize>true</visualize>
         <update_rate>30.0</update_rate>
-        <camera name="head">
-          <horizontal_fov>1.3962634</horizontal_fov>
+        <camera name="raspi_camera">
+          <horizontal_fov>1.086</horizontal_fov>
           <image>
             <width>640</width>

File: magni_description/urdf/sensors/sonar_hc-sr04.xacro (robot description, xacro)
@@ -11,5 +11,5 @@
     <link name="${name}">
       <visual>
-        <origin xyz="-0.005 0 0" rpy="${pi/2} 0 ${pi/2}" />
+        <origin xyz="-0.006 0 0" rpy="${pi/2} 0 ${pi/2}" />
         <geometry>
           <mesh filename="package://magni_description/meshes/sensors/sonar_hc-sr04.dae" />
@@ -17,5 +17,5 @@
       </visual>
       <collision>
-        <origin xyz="0.0075 0 0" rpy="0 0 0" />
+        <origin xyz="0 0 0" rpy="0 0 0" />
         <geometry>
           <box size="0.02 0.044 0.021"/>
@@ -51,5 +51,5 @@
         <!-- Gazebo-ROS interface plugin -->
         <plugin filename="libgazebo_ros_range.so" name="gazebo_ros_range">
-          <gaussianNoise>0.005</gaussianNoise>
+          <gaussianNoise>0.015</gaussianNoise>
           <alwaysOn>true</alwaysOn>
           <updateRate>5</updateRate>

Commit message: basic gound track for fiducials in gazebo

File: magni_description/urdf/magni.urdf.xacro (robot description, xacro)
@@ -147,3 +147,8 @@
     </xacro:raspi_camera>
   </xacro:if>
+  <xacro:if value="${raspicam_mount == 'true_forward'}">
+    <xacro:raspi_camera name="raspicam" connected_to="base_link">
+	<origin xyz="0.10 0.06 0.095" rpy="-${7*pi/12} 0 -${pi/2}"/>
+    </xacro:raspi_camera>
+  </xacro:if>
 </robot>

Commit message: Correcting legacy translations.  Adding two new camera poses for tilted downward and for direct forward facing camera mounts

File: magni_description/urdf/magni.urdf.xacro (robot description, xacro)
@@ -137,13 +137,27 @@
   </xacro:if>
   <!-- Define raspicam based on the raspicam_mount argument -->
+  <!-- forward  Legacy tilted slightly upwards              -->
+  <!-- upward   Legacy pointing straight up                 -->
+  <!-- downward Forward and tilted 20 deg downward          -->
+  <!-- ahead    Directly facing forward with no tilt        -->
   <xacro:if value="${raspicam_mount == 'forward'}">
-    <xacro:raspi_camera name="raspicam" connected_to="base_link">
-      <origin xyz="0.035 0.085 0.14" rpy="1.15191731 0 1.5707"/>
-    </xacro:raspi_camera>
+    <xacro:raspicam>
+      <origin xyz="0.050 0.085 0.145" rpy="1.1519 0 1.5707"/>
+    </xacro:raspicam>
   </xacro:if>
   <xacro:if value="${raspicam_mount == 'upward'}">
-    <xacro:raspi_camera name="raspicam" connected_to="base_link">
-      <origin xyz="0.035 0.15 0.14" rpy="0 0 ${pi}"/>
-    </xacro:raspi_camera>
+    <xacro:raspicam>
+      <origin xyz="0.020 0.13 0.160" rpy="0 0 ${pi}"/>
+    </xacro:raspicam>
+  </xacro:if>
+  <xacro:if value="${raspicam_mount == 'downward'}">
+    <xacro:raspicam>
+      <origin xyz="0.092 0.073 0.13" rpy="0.00 1.80 0.0"/>
+    </xacro:raspicam>
+  </xacro:if>
+  <xacro:if value="${raspicam_mount == 'ahead'}">
+    <xacro:raspicam>
+      <origin xyz="0.095 0.061 0.10" rpy="0 1.5707 0"/>
+    </xacro:raspicam>
   </xacro:if>
 </robot>

Commit message: Correcting legacy translations.  Adding two new camera poses for tilted downward and for direct forward facing camera mounts

File: magni_description/urdf/magni.urdf.xacro (robot description, xacro)
@@ -148,5 +148,5 @@
   <xacro:if value="${raspicam_mount == 'upward'}">
     <xacro:raspicam>
-      <origin xyz="0.020 0.13 0.160" rpy="0 0 ${pi}"/>
+      <origin xyz="0.020 0.115 0.160" rpy="0 0 ${pi}"/>
     </xacro:raspicam>
   </xacro:if>

Commit message: Get camera position from extrinsics file if it exists
This allows for the user to adjust the actual camera position based on
extrinsic calibration.

Fixes: https://github.com/UbiquityRobotics/magni_robot/issues/100

File: magni_description/urdf/magni.urdf.xacro (robot description, xacro)
@@ -5,4 +5,6 @@
   <xacro:arg name="sonars_installed" default="true"/>
   <xacro:property name="sonars_installed" value="$(arg sonars_installed)"/>
+  <xacro:arg name="camera_extrinsics_file" default="-"/>
+  <xacro:property name="camera_extrinsics_file" value="$(arg camera_extrinsics_file)"/>
   <xacro:property name="wheel_r" value="0.1" />
   <xacro:property name="wheel_xpos" value="0.11" />
@@ -136,14 +138,26 @@
     </xacro:sonar_hc-sr04>
   </xacro:if>
-  <!-- Define raspicam based on the raspicam_mount argument -->
-  <xacro:if value="${raspicam_mount == 'forward'}">
+  <!-- If we are given an extrinsics calibration use that instead of the pre-configured pose -->
+  <xacro:if value="${camera_extrinsics_file != '-'}">
+    <xacro:property name="cam_extrinsics" value="${load_yaml(camera_extrinsics_file)}"/>
+    <xacro:property name="cam_position" value="${cam_extrinsics['position']}"/>
+    <xacro:property name="cam_orientation" value="${cam_extrinsics['orientation']}"/>
     <xacro:raspi_camera name="raspicam" connected_to="base_link">
-      <origin xyz="0.035 0.085 0.14" rpy="1.15191731 0 1.5707"/>
+      <origin xyz="${cam_position['x']} ${cam_position['y']} ${cam_position['z']}"
+        rpy="${cam_orientation['r']} ${cam_orientation['p']} ${cam_orientation['y']}"/>
     </xacro:raspi_camera>
   </xacro:if>
-  <xacro:if value="${raspicam_mount == 'upward'}">
-    <xacro:raspi_camera name="raspicam" connected_to="base_link">
-      <origin xyz="0.035 0.15 0.14" rpy="0 0 ${pi}"/>
-    </xacro:raspi_camera>
+  <xacro:if value="${camera_extrinsics_file == '-'}">
+    <!-- Define raspicam based on the raspicam_mount argument -->
+    <xacro:if value="${raspicam_mount == 'forward'}">
+      <xacro:raspi_camera name="raspicam" connected_to="base_link">
+        <origin xyz="0.035 0.085 0.14" rpy="1.15191731 0 1.5707"/>
+      </xacro:raspi_camera>
+    </xacro:if>
+    <xacro:if value="${raspicam_mount == 'upward'}">
+      <xacro:raspi_camera name="raspicam" connected_to="base_link">
+        <origin xyz="0.035 0.15 0.14" rpy="0 0 ${pi}"/>
+      </xacro:raspi_camera>
+    </xacro:if>
   </xacro:if>
 </robot>
