Commit message: Had to merge in recent extrinsics additions to urdf

File: magni_description/urdf/magni.urdf.xacro (robot description, xacro)
@@ -5,4 +5,6 @@
   <xacro:arg name="sonars_installed" default="true"/>
   <xacro:property name="sonars_installed" value="$(arg sonars_installed)"/>
+  <xacro:arg name="camera_extrinsics_file" default="-"/>
+  <xacro:property name="camera_extrinsics_file" value="$(arg camera_extrinsics_file)"/>
   <xacro:property name="wheel_r" value="0.1" />
   <xacro:property name="wheel_xpos" value="0.11" />
@@ -20,5 +22,5 @@
       </geometry>
     </visual>
-	<visual>
+        <visual>
       <origin xyz="${-wheel_xpos-0.169} 0.17 ${-wheel_r+0.09}" rpy="0 0 ${pi}" />
       <geometry>
@@ -26,5 +28,5 @@
       </geometry>
     </visual>
-	<visual>
+        <visual>
       <origin xyz="${-wheel_xpos-0.169} -0.17 ${-wheel_r+0.09}" rpy="0 0 ${pi}" />
       <geometry>
@@ -33,5 +35,5 @@
     </visual>
     <collision>
-	  <origin xyz="${-wheel_xpos} 0 ${-wheel_r+0.151}" rpy="0 0 0" />
+          <origin xyz="${-wheel_xpos} 0 ${-wheel_r+0.151}" rpy="0 0 0" />
       <geometry>
         <box size="0.398 0.268 0.160"/>
@@ -136,28 +138,40 @@
     </xacro:sonar_hc-sr04>
   </xacro:if>
-  <!-- Define raspicam based on the raspicam_mount argument -->
-  <!-- forward  Forward and tilted slightly upwards         -->
-  <!-- upward   Pointing straight up                        -->
-  <!-- downward Forward and tilted slightly downward        -->
-  <!-- ahead    Directly facing forward with no tilt        -->
-  <xacro:if value="${raspicam_mount == 'forward'}">
-    <xacro:raspicam>
-      <origin xyz="0.050 0.085 0.145" rpy="1.1519 0 1.5707"/>
-    </xacro:raspicam>
+  <!-- If we are given an extrinsics calibration use that instead of the pre-configured pose -->
+  <xacro:if value="${camera_extrinsics_file != '-'}">
+    <xacro:property name="cam_extrinsics" value="${load_yaml(camera_extrinsics_file)}"/>
+    <xacro:property name="cam_position" value="${cam_extrinsics['position']}"/>
+    <xacro:property name="cam_orientation" value="${cam_extrinsics['orientation']}"/>
+    <xacro:raspi_camera name="raspicam" connected_to="base_link">
+      <origin xyz="${cam_position['x']} ${cam_position['y']} ${cam_position['z']}"
+        rpy="${cam_orientation['r']} ${cam_orientation['p']} ${cam_orientation['y']}"/>
+    </xacro:raspi_camera>
   </xacro:if>
-  <xacro:if value="${raspicam_mount == 'upward'}">
-    <xacro:raspicam>
-      <origin xyz="0.020 0.115 0.160" rpy="0 0 ${pi}"/>
-    </xacro:raspicam>
-  </xacro:if>
-  <xacro:if value="${raspicam_mount == 'downward'}">
-    <xacro:raspicam>
-      <origin xyz="0.092 0.073 0.13" rpy="0.00 1.80 0.0"/>
-    </xacro:raspicam>
-  </xacro:if>
-  <xacro:if value="${raspicam_mount == 'ahead'}">
-    <xacro:raspicam>
-      <origin xyz="0.095 0.061 0.10" rpy="0 1.5707 0"/>
-    </xacro:raspicam>
+  <xacro:if value="${camera_extrinsics_file == '-'}">
+    <!-- Define raspicam based on the raspicam_mount argument -->
+    <!-- forward  Forward and tilted slightly upwards         -->
+    <!-- upward   Pointing straight up                        -->
+    <!-- downward Forward and tilted slightly downward        -->
+    <!-- ahead    Directly facing forward with no tilt        -->
+    <xacro:if value="${raspicam_mount == 'forward'}">
+      <xacro:raspi_camera name="raspicam" connected_to="base_link">
+        <origin xyz="0.050 0.085 0.145" rpy="1.1519 0 1.5707"/>
+      </xacro:raspi_camera>
+    </xacro:if>
+    <xacro:if value="${raspicam_mount == 'upward'}">
+      <xacro:raspi_camera name="raspicam" connected_to="base_link">
+        <origin xyz="0.020 0.115 0.160" rpy="0 0 ${pi}"/>
+      </xacro:raspi_camera>
+    </xacro:if>
+    <xacro:if value="${raspicam_mount == 'downward'}">
+      <xacro:raspi_camera name="raspicam" connected_to="base_link">
+        <origin xyz="0.092 0.073 0.13" rpy="0.00 1.80 0.0"/>
+      </xacro:raspi_camera>
+    </xacro:if>
+    <xacro:if value="${raspicam_mount == 'ahead'}">
+      <xacro:raspi_camera name="raspicam" connected_to="base_link">
+        <origin xyz="0.095 0.061 0.10" rpy="0 1.5707 0"/>
+      </xacro:raspi_camera>
+    </xacro:if>
   </xacro:if>
 </robot>

Commit message: Add new camera poses and correct 2 existing poses (#99)
* Correcting legacy translations.  Adding two new camera poses for tilted downward and for direct forward facing camera mounts

* Correcting legacy translations.  Adding two new camera poses for tilted downward and for direct forward facing camera mounts

* Change comment line but still have 4 pose choices

* Removing the qualifier of legacy from comments as that information is not required and may just be confusing

File: magni_description/urdf/magni.urdf.xacro (robot description, xacro)
@@ -150,14 +150,28 @@
   <xacro:if value="${camera_extrinsics_file == '-'}">
     <!-- Define raspicam based on the raspicam_mount argument -->
+    <!-- forward  Forward and tilted slightly upwards         -->
+    <!-- upward   Pointing straight up                        -->
+    <!-- downward Forward and tilted slightly downward        -->
+    <!-- ahead    Directly facing forward with no tilt        -->
     <xacro:if value="${raspicam_mount == 'forward'}">
       <xacro:raspi_camera name="raspicam" connected_to="base_link">
-        <origin xyz="0.035 0.085 0.14" rpy="1.15191731 0 1.5707"/>
+        <origin xyz="0.050 0.085 0.145" rpy="1.15191731 0 1.5707"/>
       </xacro:raspi_camera>
     </xacro:if>
     <xacro:if value="${raspicam_mount == 'upward'}">
       <xacro:raspi_camera name="raspicam" connected_to="base_link">
-        <origin xyz="0.035 0.15 0.14" rpy="0 0 ${pi}"/>
+        <origin xyz="0.020 0.115 0.160" rpy="0 0 ${pi}"/>
       </xacro:raspi_camera>
     </xacro:if>
+      <xacro:if value="${raspicam_mount == 'downward'}">
+        <xacro:raspicam>
+          <origin xyz="0.092 0.073 0.13" rpy="0.00 1.80 0.0"/>
+        </xacro:raspicam>
+      </xacro:if>
+      <xacro:if value="${raspicam_mount == 'ahead'}">
+        <xacro:raspicam>
+          <origin xyz="0.095 0.061 0.10" rpy="0 1.5707 0"/>
+        </xacro:raspicam>
+      </xacro:if>
   </xacro:if>
 </robot>

Commit message: move downward urdf camera pose to high mount. Add two move_basic launch parameters but they use defaults in code still with this change

File: magni_description/urdf/magni.urdf.xacro (robot description, xacro)
@@ -152,5 +152,5 @@
     <!-- forward  Forward and tilted slightly upwards         -->
     <!-- upward   Pointing straight up                        -->
-    <!-- downward Forward and tilted slightly downward        -->
+    <!-- downward High up and tilted slightly down            -->
     <!-- ahead    Directly facing forward with no tilt        -->
     <xacro:if value="${raspicam_mount == 'forward'}">
@@ -166,5 +166,6 @@
     <xacro:if value="${raspicam_mount == 'downward'}">
       <xacro:raspi_camera name="raspicam" connected_to="base_link">
-        <origin xyz="0.092 0.073 0.13" rpy="0.00 1.80 0.0"/>
+        <!-- downward High up and tilted 35 degrees downward  -->
+        <origin xyz="0.100 0.095 0.48" rpy=" -2.1800 -0.0004562 -1.57014"/>
       </xacro:raspi_camera>
     </xacro:if>

Commit message: Changing the upward pose to proper translations

File: magni_description/urdf/magni.urdf.xacro (robot description, xacro)
@@ -157,5 +157,5 @@
     <xacro:if value="${raspicam_mount == 'upward'}">
       <xacro:raspi_camera name="raspicam" connected_to="base_link">
-        <origin xyz="0.035 0.15 0.14" rpy="0 0 ${pi}"/>
+        <origin xyz="0.020 0.115 0.16" rpy="0 0 ${pi}"/>
       </xacro:raspi_camera>
     </xacro:if>

Commit message: Modify downward raspicam pose to be high up on proposed new floor follow mounting of camera.  Some tweeks to other raspicam poses of lesser importance

File: magni_description/urdf/magni.urdf.xacro (robot description, xacro)
@@ -152,26 +152,26 @@
     <!-- forward  Forward and tilted slightly upwards         -->
     <!-- upward   Pointing straight up                        -->
-    <!-- downward Forward and tilted slightly downward        -->
+    <!-- downward High on post and pointing 45 degree down    -->
     <!-- ahead    Directly facing forward with no tilt        -->
     <xacro:if value="${raspicam_mount == 'forward'}">
       <xacro:raspi_camera name="raspicam" connected_to="base_link">
-        <origin xyz="0.050 0.085 0.145" rpy="1.15191731 0 1.5707"/>
+        <origin xyz="0.050 0.085 0.135" rpy="1.15191731 0 1.5707"/>
       </xacro:raspi_camera>
     </xacro:if>
     <xacro:if value="${raspicam_mount == 'upward'}">
       <xacro:raspi_camera name="raspicam" connected_to="base_link">
-        <origin xyz="0.020 0.115 0.160" rpy="0 0 ${pi}"/>
+        <origin xyz="0.020 0.115 0.155" rpy="0 0 ${pi}"/>
       </xacro:raspi_camera>
     </xacro:if>
-      <xacro:if value="${raspicam_mount == 'downward'}">
-        <xacro:raspicam>
-          <origin xyz="0.092 0.073 0.13" rpy="0.00 1.80 0.0"/>
-        </xacro:raspicam>
-      </xacro:if>
-      <xacro:if value="${raspicam_mount == 'ahead'}">
-        <xacro:raspicam>
-          <origin xyz="0.095 0.061 0.10" rpy="0 1.5707 0"/>
-        </xacro:raspicam>
-      </xacro:if>
+    <xacro:if value="${raspicam_mount == 'downward'}">
+      <xacro:raspicam>
+        <origin xyz="0.110 0.090 0.455" rpy="3.14159 -0.7854 0.0"/>
+      </xacro:raspicam>
+    </xacro:if>
+    <xacro:if value="${raspicam_mount == 'ahead'}">
+      <xacro:raspicam>
+        <origin xyz="0.095 0.061 0.10" rpy="0 1.5707 0"/>
+      </xacro:raspicam>
+    </xacro:if>
   </xacro:if>
 </robot>

Commit message: Sync urdf to recent master numbers.    Optimize fiducial_floor_follow.launch params

File: magni_description/urdf/magni.urdf.xacro (robot description, xacro)
@@ -156,16 +156,15 @@
     <xacro:if value="${raspicam_mount == 'forward'}">
       <xacro:raspi_camera name="raspicam" connected_to="base_link">
-        <origin xyz="0.050 0.085 0.145" rpy="1.15191731 0 1.5707"/>
+        <origin xyz="0.050 0.085 0.135" rpy="1.15191731 0 1.5707"/>
       </xacro:raspi_camera>
     </xacro:if>
     <xacro:if value="${raspicam_mount == 'upward'}">
       <xacro:raspi_camera name="raspicam" connected_to="base_link">
-        <origin xyz="0.020 0.115 0.160" rpy="0 0 ${pi}"/>
+        <origin xyz="0.020 0.115 0.155" rpy="0 0 ${pi}"/>
       </xacro:raspi_camera>
     </xacro:if>
     <xacro:if value="${raspicam_mount == 'downward'}">
       <xacro:raspi_camera name="raspicam" connected_to="base_link">
-        <!-- downward High up and tilted 35 degrees downward  -->
-        <origin xyz="0.100 0.095 0.48" rpy=" -2.1800 -0.0004562 -1.57014"/>
+        <origin xyz="0.110 0.090 0.455" rpy="3.14159 -0.7854 0.0"/>
       </xacro:raspi_camera>
     </xacro:if>

Commit message: Fixing formatting issues

File: magni_description/urdf/magni.urdf.xacro (robot description, xacro)
@@ -22,5 +22,5 @@
       </geometry>
     </visual>
-        <visual>
+    <visual>
       <origin xyz="${-wheel_xpos-0.169} 0.17 ${-wheel_r+0.09}" rpy="0 0 ${pi}" />
       <geometry>
@@ -28,5 +28,5 @@
       </geometry>
     </visual>
-        <visual>
+    <visual>
       <origin xyz="${-wheel_xpos-0.169} -0.17 ${-wheel_r+0.09}" rpy="0 0 ${pi}" />
       <geometry>
@@ -35,5 +35,5 @@
     </visual>
     <collision>
-          <origin xyz="${-wheel_xpos} 0 ${-wheel_r+0.151}" rpy="0 0 0" />
+      <origin xyz="${-wheel_xpos} 0 ${-wheel_r+0.151}" rpy="0 0 0" />
       <geometry>
         <box size="0.398 0.268 0.160"/>

Commit message: updated urdf and gazebo topics to match real robot

File: magni_description/urdf/magni.urdf.xacro (robot description, xacro)
@@ -166,5 +166,5 @@
     <xacro:if value="${raspicam_mount == 'downward'}">
       <xacro:raspi_camera name="raspicam" connected_to="base_link">
-        <origin xyz="0.110 0.090 0.455" rpy="3.14159 -0.7854 0.0"/>
+        <origin xyz="0.1 0.090 0.145" rpy="3.14159 -1.25 0.0"/>
       </xacro:raspi_camera>
     </xacro:if>

File: magni_description/urdf/sensors/sonar_hc-sr04.xacro (robot description, xacro)
@@ -39,11 +39,11 @@
               <samples>5</samples>
               <resolution>1.0</resolution>
-              <min_angle>-0.24</min_angle>
-              <max_angle>0.24</max_angle>
+              <min_angle>-0.05</min_angle>
+              <max_angle>0.05</max_angle>
             </vertical>
           </scan>
           <range>
             <min>0.02</min>
-            <max>3.2</max>
+            <max>4.0</max>
             <resolution>0.01</resolution>
           </range>
@@ -54,5 +54,5 @@
           <alwaysOn>true</alwaysOn>
           <updateRate>5</updateRate>
-          <topicName>/ubiquity_sonar/${name}</topicName>
+          <topicName>/pi_sonar/${name}</topicName>
           <frameName>${name}</frameName>
           <fov>0.5</fov>

Commit message: added optional lidar

File: magni_description/urdf/magni.urdf.xacro (robot description, xacro)
@@ -7,4 +7,6 @@
   <xacro:arg name="camera_extrinsics_file" default="-"/>
   <xacro:property name="camera_extrinsics_file" value="$(arg camera_extrinsics_file)"/>
+  <xacro:arg name="lidar_installed" default="false"/>
+  <xacro:property name="lidar_installed" value="$(arg lidar_installed)"/>
   <xacro:property name="wheel_r" value="0.1" />
   <xacro:property name="wheel_xpos" value="0.11" />
@@ -14,4 +16,5 @@
   <xacro:include filename="$(find magni_description)/urdf/sensors/sonar_hc-sr04.xacro" />
   <xacro:include filename="$(find magni_description)/urdf/sensors/raspi_camera.xacro" />
+  <xacro:include filename="$(find magni_description)/urdf/sensors/hokuyo_lidar.xacro" />
   <!-- Robot base_link -->
   <link name="base_link">
@@ -175,3 +178,8 @@
     </xacro:if>
   </xacro:if>
+ <xacro:if value="${lidar_installed}">
+    <xacro:hokuyo_lidar name="laser" connected_to="base_link">
+      <origin xyz="0 0.0 0.2" rpy="0 0 0"/>
+    </xacro:hokuyo_lidar>
+  </xacro:if>
 </robot>

File: magni_description/urdf/sensors/raspi_camera.xacro (robot description, xacro)
@@ -52,5 +52,5 @@
           <updateRate>0.0</updateRate>
           <cameraName>${name}</cameraName>
-          <imageTopicName>/${name}_node/image/compressed</imageTopicName>
+          <imageTopicName>/${name}_node/image</imageTopicName>
           <cameraInfoTopicName>/${name}_node/camera_info</cameraInfoTopicName>
           <frameName>${name}</frameName>

Commit message: Fixes yaml parsing into magni.urdf.xacro

File: magni_description/urdf/magni.urdf.xacro (robot description, xacro)
@@ -144,6 +144,6 @@
     <xacro:property name="cam_orientation" value="${cam_extrinsics['orientation']}"/>
     <xacro:raspi_camera name="raspicam" connected_to="base_link">
-      <origin xyz="${cam_position['x']} ${cam_position['y']} ${cam_position['z']}"
-        rpy="${cam_orientation['r']} ${cam_orientation['p']} ${cam_orientation['y']}"/>
+      <origin xyz="${cam_position[0]} ${cam_position[1]} ${cam_position[2]}"
+        rpy="${cam_orientation[0]} ${cam_orientation[1]} ${cam_orientation[2]}"/>
     </xacro:raspi_camera>
   </xacro:if>

Commit message: Camera sensor link fix

File: magni_description/urdf/magni.urdf.xacro (robot description, xacro)
@@ -159,24 +159,25 @@
     <xacro:if value="${raspicam_mount == 'forward'}">
       <xacro:raspi_camera name="raspicam" connected_to="base_link">
-        <origin xyz="0.050 0.085 0.135" rpy="1.15191731 0 1.5707"/>
+        <origin xyz="0.050 0.085 0.135" rpy="0 ${-pi/2 - 1.15191731} ${pi}"/>
       </xacro:raspi_camera>
     </xacro:if>
     <xacro:if value="${raspicam_mount == 'upward'}">
       <xacro:raspi_camera name="raspicam" connected_to="base_link">
-        <origin xyz="0.020 0.115 0.155" rpy="0 0 ${pi}"/>
+        <origin xyz="0.020 0.115 0.155" rpy="0 ${-pi/2} ${-pi/2}"/>
       </xacro:raspi_camera>
     </xacro:if>
     <xacro:if value="${raspicam_mount == 'downward'}">
       <xacro:raspi_camera name="raspicam" connected_to="base_link">
-        <origin xyz="0.1 0.090 0.145" rpy="3.14159 -1.25 0.0"/>
+        <origin xyz="0.1 0.090 0.145" rpy="${-pi/2} ${pi/2 - 1.25} 0.0"/>
       </xacro:raspi_camera>
     </xacro:if>
     <xacro:if value="${raspicam_mount == 'ahead'}">
       <xacro:raspi_camera name="raspicam" connected_to="base_link">
-        <origin xyz="0.095 0.061 0.10" rpy="0 1.5707 0"/>
+        <origin xyz="0.095 0.061 0.10" rpy="${pi/2} 0 0"/>
       </xacro:raspi_camera>
     </xacro:if>
   </xacro:if>
- <xacro:if value="${lidar_installed}">
+  <!-- Define lidar -->
+  <xacro:if value="${lidar_installed}">
     <xacro:hokuyo_lidar name="laser" connected_to="base_link">
       <origin xyz="0 0.0 0.2" rpy="0 0 0"/>

File: magni_description/urdf/sensors/raspi_camera.xacro (robot description, xacro)
@@ -11,5 +11,5 @@
     <link name="${name}">
       <visual>
-        <origin xyz="0 0 0" rpy="${pi/2} 0 0" />
+        <origin xyz="0 0 0" rpy="0 0 ${-pi/2}" />
         <geometry>
           <mesh filename="package://magni_description/meshes/sensors/raspi_camera.dae" />
@@ -23,13 +23,13 @@
       </collision>
     </link>
-    <!-- Additional link for camera Gazebo sensor to orient camera direction (it is used only for Gazebo simulation) -->
-    <link name="${name}_gazebo_sensor"/>
-    <joint name="${name}_gazebo_sensor_joint" type="fixed">
+    <!-- Additional link for camera sensor -->
+    <link name="${name}_sensor"/>
+    <joint name="${name}_sensor_joint" type="fixed">
       <parent link="${name}"/>
-      <child link="${name}_gazebo_sensor"/>
-      <origin xyz="0 0 0.012" rpy="${pi/2} ${-pi/2} 0" />
+      <child link="${name}_sensor"/>
+      <origin xyz="0.005 0 0" rpy="${-pi/2} 0 ${-pi/2}" />
     </joint>
-    <!-- Gazebo sensor plugin -->
-    <gazebo reference="${name}_gazebo_sensor">
+    <!-- Gazebo sensor plugin. Gazebo sensor is attached to camera link (${name}) but publishes its messages to ${name}_sensor frame. -->
+    <gazebo reference="${name}">
       <sensor type="camera" name="camera1">
         <visualize>false</visualize>
@@ -51,8 +51,8 @@
           <alwaysOn>true</alwaysOn>
           <updateRate>0.0</updateRate>
-          <cameraName>${name}</cameraName>
-          <imageTopicName>/${name}_node/image</imageTopicName>
-          <cameraInfoTopicName>/${name}_node/camera_info</cameraInfoTopicName>
-          <frameName>${name}</frameName>
+          <cameraName></cameraName>
+          <imageTopicName>${name}_node/image</imageTopicName>
+          <cameraInfoTopicName>${name}_node/camera_info</cameraInfoTopicName>
+          <frameName>${name}_sensor</frameName>
           <hackBaseline>0.07</hackBaseline>
           <distortionK1>0.0</distortionK1>

Commit message: Update camera 'Ahead' position to straight vertically

File: magni_description/urdf/magni.urdf.xacro (robot description, xacro)
@@ -174,5 +174,5 @@
     <xacro:if value="${raspicam_mount == 'ahead'}">
       <xacro:raspi_camera name="raspicam" connected_to="base_link">
-        <origin xyz="0.095 0.061 0.10" rpy="${pi/2} 0 0"/>
+        <origin xyz="0.095 0.061 0.10" rpy="0 0 0"/>
       </xacro:raspi_camera>
     </xacro:if>

Commit message: innitial xml write example for camera

File: magni_description/urdf/magni.urdf.xacro (robot description, xacro)
@@ -1,12 +1,22 @@
 <?xml version="1.0"?>
 <robot xmlns:xacro="http://wiki.ros.org/xacro" name="magni">
-  <xacro:arg name="raspicam_mount" default="forward"/>
-  <xacro:property name="raspicam_mount" value="$(arg raspicam_mount)"/>
   <xacro:arg name="sonars_installed" default="true"/>
   <xacro:property name="sonars_installed" value="$(arg sonars_installed)"/>
-  <xacro:arg name="camera_extrinsics_file" default="-"/>
-  <xacro:property name="camera_extrinsics_file" value="$(arg camera_extrinsics_file)"/>
+  <xacro:arg name="camera_installed" default="true"/>
+  <xacro:property name="camera_installed" value="$(arg camera_installed)"/>
   <xacro:arg name="lidar_installed" default="false"/>
   <xacro:property name="lidar_installed" value="$(arg lidar_installed)"/>
+  <xacro:arg name="cam_ext_x" default="0.0"/>
+  <xacro:arg name="cam_ext_y" default="0.0"/>
+  <xacro:arg name="cam_ext_z" default="0.0"/>
+  <xacro:arg name="cam_ext_roll" default="0.0"/>
+  <xacro:arg name="cam_ext_pitch" default="0.0"/>
+  <xacro:arg name="cam_ext_yaw" default="0.0"/>
+  <xacro:property name="cam_ext_x" value="$(arg cam_ext_x)"/>
+  <xacro:property name="cam_ext_y" value="$(arg cam_ext_y)"/>
+  <xacro:property name="cam_ext_z" value="$(arg cam_ext_z)"/>
+  <xacro:property name="cam_ext_roll" value="$(arg cam_ext_roll)"/>
+  <xacro:property name="cam_ext_pitch" value="$(arg cam_ext_pitch)"/>
+  <xacro:property name="cam_ext_yaw" value="$(arg cam_ext_yaw)"/>
   <xacro:property name="wheel_r" value="0.1" />
   <xacro:property name="wheel_xpos" value="0.11" />
@@ -141,40 +151,8 @@
     </xacro:sonar_hc-sr04>
   </xacro:if>
-  <!-- If we are given an extrinsics calibration use that instead of the pre-configured pose -->
-  <xacro:if value="${camera_extrinsics_file != '-'}">
-    <xacro:property name="cam_extrinsics" value="${load_yaml(camera_extrinsics_file)}"/>
-    <xacro:property name="cam_position" value="${cam_extrinsics['position']}"/>
-    <xacro:property name="cam_orientation" value="${cam_extrinsics['orientation']}"/>
+  <xacro:if value="${camera_installed}">
     <xacro:raspi_camera name="raspicam" connected_to="base_link">
-      <origin xyz="${cam_position[0]} ${cam_position[1]} ${cam_position[2]}"
-        rpy="${cam_orientation[0]} ${cam_orientation[1]} ${cam_orientation[2]}"/>
+      <origin xyz="${cam_ext_x} ${cam_ext_y} ${cam_ext_z}" rpy="${cam_ext_roll} ${cam_ext_pitch} ${cam_ext_yaw}"/>
     </xacro:raspi_camera>
-  </xacro:if>
-  <xacro:if value="${camera_extrinsics_file == '-'}">
-    <!-- Define raspicam based on the raspicam_mount argument -->
-    <!-- forward  Forward and tilted slightly upwards         -->
-    <!-- upward   Pointing straight up                        -->
-    <!-- downward High on post and pointing 45 degree down    -->
-    <!-- ahead    Directly facing forward with no tilt        -->
-    <xacro:if value="${raspicam_mount == 'forward'}">
-      <xacro:raspi_camera name="raspicam" connected_to="base_link">
-        <origin xyz="0.050 0.085 0.135" rpy="0 ${-pi/2 - 1.15191731} ${pi}"/>
-      </xacro:raspi_camera>
-    </xacro:if>
-    <xacro:if value="${raspicam_mount == 'upward'}">
-      <xacro:raspi_camera name="raspicam" connected_to="base_link">
-        <origin xyz="0.020 0.115 0.155" rpy="0 ${-pi/2} ${-pi/2}"/>
-      </xacro:raspi_camera>
-    </xacro:if>
-    <xacro:if value="${raspicam_mount == 'downward'}">
-      <xacro:raspi_camera name="raspicam" connected_to="base_link">
-        <origin xyz="0.1 0.090 0.145" rpy="${-pi/2} ${pi/2 - 1.25} 0.0"/>
-      </xacro:raspi_camera>
-    </xacro:if>
-    <xacro:if value="${raspicam_mount == 'ahead'}">
-      <xacro:raspi_camera name="raspicam" connected_to="base_link">
-        <origin xyz="0.095 0.061 0.10" rpy="0 0 0"/>
-      </xacro:raspi_camera>
-    </xacro:if>
   </xacro:if>
   <!-- Define lidar -->
