Commit message: Fist testing of launch file generation on the robot

File: magni_description/urdf/magni.urdf.xacro (robot description, xacro)
@@ -7,16 +7,16 @@
   <xacro:arg name="lidar_installed" default="false"/>
   <xacro:property name="lidar_installed" value="$(arg lidar_installed)"/>
-  <xacro:arg name="cam_ext_x" default="0.0"/>
-  <xacro:arg name="cam_ext_y" default="0.0"/>
-  <xacro:arg name="cam_ext_z" default="0.0"/>
-  <xacro:arg name="cam_ext_roll" default="0.0"/>
-  <xacro:arg name="cam_ext_pitch" default="0.0"/>
-  <xacro:arg name="cam_ext_yaw" default="0.0"/>
-  <xacro:property name="cam_ext_x" value="$(arg cam_ext_x)"/>
-  <xacro:property name="cam_ext_y" value="$(arg cam_ext_y)"/>
-  <xacro:property name="cam_ext_z" value="$(arg cam_ext_z)"/>
-  <xacro:property name="cam_ext_roll" value="$(arg cam_ext_roll)"/>
-  <xacro:property name="cam_ext_pitch" value="$(arg cam_ext_pitch)"/>
-  <xacro:property name="cam_ext_yaw" value="$(arg cam_ext_yaw)"/>
+  <xacro:arg name="camera_extr_x" default="0.0"/>
+  <xacro:arg name="camera_extr_y" default="0.0"/>
+  <xacro:arg name="camera_extr_z" default="0.0"/>
+  <xacro:arg name="camera_extr_roll" default="0.0"/>
+  <xacro:arg name="camera_extr_pitch" default="0.0"/>
+  <xacro:arg name="camera_extr_yaw" default="0.0"/>
+  <xacro:arg name="lidar_extr_x" default="0.0"/>
+  <xacro:arg name="lidar_extr_y" default="0.0"/>
+  <xacro:arg name="lidar_extr_z" default="0.0"/>
+  <xacro:arg name="lidar_extr_roll" default="0.0"/>
+  <xacro:arg name="lidar_extr_pitch" default="0.0"/>
+  <xacro:arg name="lidar_extr_yaw" default="0.0"/>
   <xacro:property name="wheel_r" value="0.1" />
   <xacro:property name="wheel_xpos" value="0.11" />
@@ -153,5 +153,5 @@
   <xacro:if value="${camera_installed}">
     <xacro:raspi_camera name="raspicam" connected_to="base_link">
-      <origin xyz="${cam_ext_x} ${cam_ext_y} ${cam_ext_z}" rpy="${cam_ext_roll} ${cam_ext_pitch} ${cam_ext_yaw}"/>
+      <origin xyz="$(arg camera_extr_x) $(arg camera_extr_y) $(arg camera_extr_z)" rpy="$(arg camera_extr_roll) $(arg camera_extr_pitch) $(arg camera_extr_yaw)"/>
     </xacro:raspi_camera>
   </xacro:if>
@@ -159,5 +159,5 @@
   <xacro:if value="${lidar_installed}">
     <xacro:hokuyo_lidar name="laser" connected_to="base_link">
-      <origin xyz="0 0.0 0.2" rpy="0 0 0"/>
+      <origin xyz="$(arg lidar_extr_x) $(arg lidar_extr_y) $(arg lidar_extr_z)" rpy="$(arg lidar_extr_roll) $(arg lidar_extr_pitch) $(arg lidar_extr_yaw)"/>
     </xacro:hokuyo_lidar>
   </xacro:if>

Commit message: extrinsics yaml file is loaded directly into urdf

File: magni_description/urdf/magni.urdf.xacro (robot description, xacro)
@@ -19,4 +19,8 @@
   <xacro:arg name="lidar_extr_pitch" default="0.0"/>
   <xacro:arg name="lidar_extr_yaw" default="0.0"/>
+  <xacro:arg name="camera_extrinsics_file" default=""/>
+  <xacro:property name="camera_extrinsics_file" value="$(arg camera_extrinsics_file)"/>
+  <xacro:arg name="lidar_extrinsics_file" default=""/>
+  <xacro:property name="lidar_extrinsics_file" value="$(arg lidar_extrinsics_file)"/>
   <xacro:property name="wheel_r" value="0.1" />
   <xacro:property name="wheel_xpos" value="0.11" />
@@ -151,13 +155,23 @@
     </xacro:sonar_hc-sr04>
   </xacro:if>
-  <xacro:if value="${camera_installed}">
+  <!-- <xacro:if value="${camera_installed}">
     <xacro:raspi_camera name="raspicam" connected_to="base_link">
       <origin xyz="$(arg camera_extr_x) $(arg camera_extr_y) $(arg camera_extr_z)" rpy="$(arg camera_extr_roll) $(arg camera_extr_pitch) $(arg camera_extr_yaw)"/>
     </xacro:raspi_camera>
+  </xacro:if> -->
+  <!-- Define camera -->
+  <xacro:if value="${camera_extrinsics_file != ''}">
+    <xacro:property name="cam_extrinsics" value="${load_yaml(camera_extrinsics_file)}"/>
+    <xacro:raspi_camera name="raspicam" connected_to="base_link">
+      <origin xyz="${cam_extrinsics['x']} ${cam_extrinsics['y']} ${cam_extrinsics['z']}"
+        rpy="${cam_extrinsics['roll']} ${cam_extrinsics['pitch']} ${cam_extrinsics['yaw']}"/>
+    </xacro:raspi_camera>
   </xacro:if>
-  <!-- Define lidar -->
-  <xacro:if value="${lidar_installed}">
+  <!-- Define Lidar -->
+  <xacro:if value="${lidar_extrinsics_file != ''}">
+    <xacro:property name="lidar_extrinsics" value="${load_yaml(lidar_extrinsics_file)}"/>
     <xacro:hokuyo_lidar name="laser" connected_to="base_link">
-      <origin xyz="$(arg lidar_extr_x) $(arg lidar_extr_y) $(arg lidar_extr_z)" rpy="$(arg lidar_extr_roll) $(arg lidar_extr_pitch) $(arg lidar_extr_yaw)"/>
+      <origin xyz="${lidar_extrinsics['x']} ${lidar_extrinsics['y']} ${lidar_extrinsics['z']}"
+        rpy="${lidar_extrinsics['roll']} ${lidar_extrinsics['pitch']} ${lidar_extrinsics['yaw']}"/>
     </xacro:hokuyo_lidar>
   </xacro:if>

Commit message: removed extrinsics by each coordinate in urdf

File: magni_description/urdf/magni.urdf.xacro (robot description, xacro)
@@ -3,20 +3,4 @@
   <xacro:arg name="sonars_installed" default="true"/>
   <xacro:property name="sonars_installed" value="$(arg sonars_installed)"/>
-  <xacro:arg name="camera_installed" default="true"/>
-  <xacro:property name="camera_installed" value="$(arg camera_installed)"/>
-  <xacro:arg name="lidar_installed" default="false"/>
-  <xacro:property name="lidar_installed" value="$(arg lidar_installed)"/>
-  <xacro:arg name="camera_extr_x" default="0.0"/>
-  <xacro:arg name="camera_extr_y" default="0.0"/>
-  <xacro:arg name="camera_extr_z" default="0.0"/>
-  <xacro:arg name="camera_extr_roll" default="0.0"/>
-  <xacro:arg name="camera_extr_pitch" default="0.0"/>
-  <xacro:arg name="camera_extr_yaw" default="0.0"/>
-  <xacro:arg name="lidar_extr_x" default="0.0"/>
-  <xacro:arg name="lidar_extr_y" default="0.0"/>
-  <xacro:arg name="lidar_extr_z" default="0.0"/>
-  <xacro:arg name="lidar_extr_roll" default="0.0"/>
-  <xacro:arg name="lidar_extr_pitch" default="0.0"/>
-  <xacro:arg name="lidar_extr_yaw" default="0.0"/>
   <xacro:arg name="camera_extrinsics_file" default=""/>
   <xacro:property name="camera_extrinsics_file" value="$(arg camera_extrinsics_file)"/>

Commit message: Added default cam positions, prettier printing

File: magni_description/urdf/magni.urdf.xacro (robot description, xacro)
@@ -139,9 +139,4 @@
     </xacro:sonar_hc-sr04>
   </xacro:if>
-  <!-- <xacro:if value="${camera_installed}">
-    <xacro:raspi_camera name="raspicam" connected_to="base_link">
-      <origin xyz="$(arg camera_extr_x) $(arg camera_extr_y) $(arg camera_extr_z)" rpy="$(arg camera_extr_roll) $(arg camera_extr_pitch) $(arg camera_extr_yaw)"/>
-    </xacro:raspi_camera>
-  </xacro:if> -->
   <!-- Define camera -->
   <xacro:if value="${camera_extrinsics_file != ''}">

Commit message: added ur50 lidar to mesh

File: magni_description/urdf/magni.urdf.xacro (robot description, xacro)
@@ -14,5 +14,5 @@
   <xacro:include filename="$(find magni_description)/urdf/sensors/sonar_hc-sr04.xacro" />
   <xacro:include filename="$(find magni_description)/urdf/sensors/raspi_camera.xacro" />
-  <xacro:include filename="$(find magni_description)/urdf/sensors/hokuyo_lidar.xacro" />
+  <xacro:include filename="$(find magni_description)/urdf/sensors/ur50_lidar.xacro" />
   <!-- Robot base_link -->
   <link name="base_link">
@@ -150,8 +150,8 @@
   <xacro:if value="${lidar_extrinsics_file != ''}">
     <xacro:property name="lidar_extrinsics" value="${load_yaml(lidar_extrinsics_file)}"/>
-    <xacro:hokuyo_lidar name="laser" connected_to="base_link">
+    <xacro:ur50_lidar name="laser" connected_to="base_link">
       <origin xyz="${lidar_extrinsics['x']} ${lidar_extrinsics['y']} ${lidar_extrinsics['z']}"
         rpy="${lidar_extrinsics['roll']} ${lidar_extrinsics['pitch']} ${lidar_extrinsics['yaw']}"/>
-    </xacro:hokuyo_lidar>
+    </xacro:ur50_lidar>
   </xacro:if>
 </robot>

File: magni_description/urdf/sensors/ur50_lidar.xacro (robot description, xacro)
@@ -1,5 +1,5 @@
 <?xml version="1.0" encoding="utf-8"?>
 <robot xmlns:xacro="http://wiki.ros.org/xacro">
-  <xacro:macro name="hokuyo_lidar" params="name:='' connected_to:='' *origin">
+  <xacro:macro name="ur50_lidar" params="name:='' connected_to:='' *origin">
   <xacro:unless value="${connected_to == ''}">
     <joint name="${name}_joint" type="fixed">
@@ -13,5 +13,5 @@
       <origin xyz="0 0 0" rpy="0 0 0" />
       <geometry>
-        <mesh filename="package://magni_description/meshes/sensors/hokuyo.dae" />
+        <mesh filename="package://magni_description/meshes/sensors/ur50_lidar.dae" />
       </geometry>
     </visual>

Commit message: added visual and collision for shell and tower

File: magni_description/urdf/magni.urdf.xacro (robot description, xacro)
@@ -62,4 +62,53 @@
       <origin xyz="-0.15 0 0.03" rpy="0 0 0" />
     </xacro:box_inertial_with_origin>
+   <!-- Robot Tower -->
+    <visual>
+      <origin xyz="0 0 0" rpy="0 0 0" />
+      <geometry>
+        <mesh filename="package://magni_description/meshes/magni_tower.dae" />
+      </geometry>
+    </visual>
+    <!-- Collision for screen -->
+    <collision>
+      <origin xyz="0.115 0 0.635" rpy="0 0.56 0" />
+      <geometry>
+        <box size="0.04 0.23 0.15"/>
+      </geometry>
+    </collision>
+    <!-- Collision for tower -->
+    <collision>
+      <origin xyz="0.08 0 0.37" rpy="0 0 0" />
+      <geometry>
+        <box size="0.06 0.24 0.40"/>
+      </geometry>
+    </collision>
+    <!-- Robot shell -->
+    <visual>
+      <origin xyz="0 0 0" rpy="0 0 0" />
+      <geometry>
+        <mesh filename="package://magni_description/meshes/magni_shell.dae" />
+      </geometry>
+    </visual>
+    <!-- Collision for shell -->
+    <collision>
+      <origin xyz="-0.11 0 0.07" rpy="0 0.0 0" />
+      <geometry>
+        <box size="0.45 0.33 0.2"/>
+      </geometry>
+    </collision>
+    <!-- Lower shelf -->
+    <collision>
+      <origin xyz="-0.18 0 0.2" rpy="0 0 0" />
+      <geometry>
+        <box size="0.35 0.408 0.005"/>
+      </geometry>
+    </collision>
+    <!-- Upper shelf -->
+    <collision>
+      <origin xyz="-0.1 0 0.53" rpy="0 0 0" />
+      <geometry>
+        <box size="0.32 0.42 0.02"/>
+      </geometry>
+    </collision>
   </link>
   <!-- Fixed offset from the floor to the center of the wheels -->

Commit message: tower and shell positions for gazebo in launches

File: magni_description/urdf/magni.urdf.xacro (robot description, xacro)
@@ -3,4 +3,8 @@
   <xacro:arg name="sonars_installed" default="true"/>
   <xacro:property name="sonars_installed" value="$(arg sonars_installed)"/>
+  <xacro:arg name="shell_installed" default="false"/>
+  <xacro:property name="shell_installed" value="$(arg shell_installed)"/>
+  <xacro:arg name="tower_installed" default="false"/>
+  <xacro:property name="tower_installed" value="$(arg tower_installed)"/>
   <xacro:arg name="camera_extrinsics_file" default=""/>
   <xacro:property name="camera_extrinsics_file" value="$(arg camera_extrinsics_file)"/>
@@ -62,53 +66,57 @@
       <origin xyz="-0.15 0 0.03" rpy="0 0 0" />
     </xacro:box_inertial_with_origin>
-   <!-- Robot Tower -->
-    <visual>
-      <origin xyz="0 0 0" rpy="0 0 0" />
-      <geometry>
-        <mesh filename="package://magni_description/meshes/magni_tower.dae" />
-      </geometry>
-    </visual>
-    <!-- Collision for screen -->
-    <collision>
-      <origin xyz="0.115 0 0.635" rpy="0 0.56 0" />
-      <geometry>
-        <box size="0.04 0.23 0.15"/>
-      </geometry>
-    </collision>
-    <!-- Collision for tower -->
-    <collision>
-      <origin xyz="0.08 0 0.37" rpy="0 0 0" />
-      <geometry>
-        <box size="0.06 0.24 0.40"/>
-      </geometry>
-    </collision>
-    <!-- Robot shell -->
-    <visual>
-      <origin xyz="0 0 0" rpy="0 0 0" />
-      <geometry>
-        <mesh filename="package://magni_description/meshes/magni_shell.dae" />
-      </geometry>
-    </visual>
-    <!-- Collision for shell -->
-    <collision>
-      <origin xyz="-0.11 0 0.07" rpy="0 0.0 0" />
-      <geometry>
-        <box size="0.45 0.33 0.2"/>
-      </geometry>
-    </collision>
-    <!-- Lower shelf -->
-    <collision>
-      <origin xyz="-0.18 0 0.2" rpy="0 0 0" />
-      <geometry>
-        <box size="0.35 0.408 0.005"/>
-      </geometry>
-    </collision>
-    <!-- Upper shelf -->
-    <collision>
-      <origin xyz="-0.1 0 0.53" rpy="0 0 0" />
-      <geometry>
-        <box size="0.32 0.42 0.02"/>
-      </geometry>
-    </collision>
+    <xacro:if value="${tower_installed}">
+      <!-- Robot Tower -->
+      <visual>
+        <origin xyz="0 0 0.005" rpy="0 0 0" />
+        <geometry>
+          <mesh filename="package://magni_description/meshes/magni_tower.dae" />
+        </geometry>
+      </visual>
+      <!-- Collision for screen -->
+      <collision>
+        <origin xyz="0.115 0 0.635" rpy="0 0.56 0" />
+        <geometry>
+          <box size="0.04 0.23 0.15"/>
+        </geometry>
+      </collision>
+      <!-- Collision for tower -->
+      <collision>
+        <origin xyz="0.08 0 0.37" rpy="0 0 0" />
+        <geometry>
+          <box size="0.06 0.24 0.40"/>
+        </geometry>
+      </collision>
+    </xacro:if>
+    <xacro:if value="${shell_installed}">
+      <!-- Robot shell -->
+      <visual>
+        <origin xyz="0 0 0.005" rpy="0 0 0" />
+        <geometry>
+          <mesh filename="package://magni_description/meshes/magni_shell.dae" />
+        </geometry>
+      </visual>
+      <!-- Collision for shell -->
+      <collision>
+        <origin xyz="-0.11 0 0.07" rpy="0 0.0 0" />
+        <geometry>
+          <box size="0.45 0.33 0.2"/>
+        </geometry>
+      </collision>
+      <!-- Lower shelf -->
+      <collision>
+        <origin xyz="-0.18 0 0.2" rpy="0 0 0" />
+        <geometry>
+          <box size="0.35 0.408 0.005"/>
+        </geometry>
+      </collision>
+      <!-- Upper shelf -->
+      <collision>
+        <origin xyz="-0.1 0 0.53" rpy="0 0 0" />
+        <geometry>
+          <box size="0.32 0.42 0.02"/>
+        </geometry>
+      </collision>
+    </xacro:if>
   </link>
   <!-- Fixed offset from the floor to the center of the wheels -->

Commit message: added laser filter and tower&shell to default robot.yaml

File: magni_description/urdf/magni.urdf.xacro (robot description, xacro)
@@ -81,9 +81,30 @@
         </geometry>
       </collision>
-      <!-- Collision for tower -->
+      <!-- Collision for tower vertical-->
       <collision>
         <origin xyz="0.08 0 0.37" rpy="0 0 0" />
         <geometry>
           <box size="0.06 0.24 0.40"/>
+        </geometry>
+      </collision>
+      <!-- Collision for tower horizontal -->
+      <collision>
+        <origin xyz="-0.1 0 0.18" rpy="0 0 0" />
+        <geometry>
+          <box size="0.42 0.24 0.03"/>
+        </geometry>
+      </collision>
+      <!-- Lower shelf -->
+      <collision>
+        <origin xyz="-0.18 0 0.2" rpy="0 0 0" />
+        <geometry>
+          <box size="0.35 0.408 0.005"/>
+        </geometry>
+      </collision>
+      <!-- Upper shelf -->
+      <collision>
+        <origin xyz="-0.1 0 0.53" rpy="0 0 0" />
+        <geometry>
+          <box size="0.32 0.42 0.02"/>
         </geometry>
       </collision>
@@ -99,21 +120,7 @@
       <!-- Collision for shell -->
       <collision>
-        <origin xyz="-0.11 0 0.07" rpy="0 0.0 0" />
-        <geometry>
-          <box size="0.45 0.33 0.2"/>
-        </geometry>
-      </collision>
-      <!-- Lower shelf -->
-      <collision>
-        <origin xyz="-0.18 0 0.2" rpy="0 0 0" />
-        <geometry>
-          <box size="0.35 0.408 0.005"/>
-        </geometry>
-      </collision>
-      <!-- Upper shelf -->
-      <collision>
-        <origin xyz="-0.1 0 0.53" rpy="0 0 0" />
-        <geometry>
-          <box size="0.32 0.42 0.02"/>
+        <origin xyz="-0.175 0 0.07" rpy="0 0.0 0" />
+        <geometry>
+          <box size="0.3 0.33 0.2"/>
         </geometry>
       </collision>

Commit message: gps extrinsics

File: magni_description/urdf/magni.urdf.xacro (robot description, xacro)
@@ -11,4 +11,6 @@
   <xacro:arg name="lidar_extrinsics_file" default=""/>
   <xacro:property name="lidar_extrinsics_file" value="$(arg lidar_extrinsics_file)"/>
+  <xacro:arg name="gps_extrinsics_file" default=""/>
+  <xacro:property name="gps_extrinsics_file" value="$(arg gps_extrinsics_file)"/>
   <xacro:property name="wheel_r" value="0.1" />
   <xacro:property name="wheel_xpos" value="0.11" />
@@ -219,3 +221,14 @@
     </xacro:ur50_lidar>
   </xacro:if>
+  <!-- Define GNSS -->
+  <xacro:if value="${gps_extrinsics_file != ''}">
+    <xacro:property name="gps_extrinsics" value="${load_yaml(gps_extrinsics_file)}"/>
+    <link name="gps"/>
+    <joint name="gps_joint" type="fixed">
+      <parent link="base_link"/>
+      <child link="gps"/>
+      <origin xyz="${gps_extrinsics['x']} ${gps_extrinsics['y']} ${gps_extrinsics['z']}"
+        rpy="${gps_extrinsics['roll']} ${gps_extrinsics['pitch']} ${gps_extrinsics['yaw']}"/>
+    </joint>
+  </xacro:if>
 </robot>

Commit message: Added ros2_control block

File: magni_description/urdf/magni.urdf.xacro (robot description, xacro)
@@ -219,3 +219,21 @@
     </xacro:ur50_lidar>
   </xacro:if>
+ <!-- ROS 2 Control block -->
+  <ros2_control name="ubiquity_motor_ros2/MotorHardware" type="system">
+    <hardware>
+      <plugin>ubiquity_motor_ros2/MotorHardware</plugin>
+    </hardware>
+    <joint name="left_wheel_joint">
+      <command_interface name="velocity"/>
+      <state_interface name="position"/>
+      <state_interface name="velocity"/>
+      <state_interface name="effort"/>
+    </joint>
+    <joint name="right_wheel_joint">
+      <command_interface name="velocity"/>
+      <state_interface name="position"/>
+      <state_interface name="velocity"/>
+      <state_interface name="effort"/>
+    </joint>
+  </ros2_control>
 </robot>

Commit message: urdf fixes for Jazzy

File: magni_description/urdf/magni.urdf.xacro (robot description, xacro)
@@ -205,5 +205,5 @@
   <!-- Define camera -->
   <xacro:if value="${camera_extrinsics_file != ''}">
-    <xacro:property name="cam_extrinsics" value="${load_yaml(camera_extrinsics_file)}"/>
+    <xacro:property name="cam_extrinsics" value="${xacro.load_yaml(camera_extrinsics_file)}"/>
     <xacro:raspi_camera name="raspicam" connected_to="base_link">
       <origin xyz="${cam_extrinsics['x']} ${cam_extrinsics['y']} ${cam_extrinsics['z']}"
@@ -213,5 +213,5 @@
   <!-- Define Lidar -->
   <xacro:if value="${lidar_extrinsics_file != ''}">
-    <xacro:property name="lidar_extrinsics" value="${load_yaml(lidar_extrinsics_file)}"/>
+    <xacro:property name="lidar_extrinsics" value="${xacro.load_yaml(lidar_extrinsics_file)}"/>
     <xacro:ur50_lidar name="laser" connected_to="base_link">
       <origin xyz="${lidar_extrinsics['x']} ${lidar_extrinsics['y']} ${lidar_extrinsics['z']}"

Commit message: added light sensor mesh and edited Magni urdf with light sesnsor

File: magni_description/urdf/magni.urdf.xacro (robot description, xacro)
@@ -19,4 +19,5 @@
   <xacro:include filename="$(find magni_description)/urdf/sensors/raspi_camera.xacro" />
   <xacro:include filename="$(find magni_description)/urdf/sensors/ur50_lidar.xacro" />
+  <xacro:include filename="$(find magni_description)/urdf/sensors/light_sensor.xacro" />
   <!-- Robot base_link -->
   <link name="base_link">
@@ -219,3 +220,8 @@
     </xacro:ur50_lidar>
   </xacro:if>
+  <!-- Define light sensor -->
+  <xacro:light_sensor name="light_sensor" connected_to="base_link">
+    <origin xyz="0.37 0 0"
+      rpy="0 0 0"/>
+  </xacro:light_sensor>
 </robot>

Commit message: added light sensor mesh and edited Magni urdf with light sesnsor

File: magni_description/urdf/magni.urdf.xacro (robot description, xacro)
@@ -21,4 +21,5 @@
   <xacro:include filename="$(find magni_description)/urdf/sensors/raspi_camera.xacro" />
   <xacro:include filename="$(find magni_description)/urdf/sensors/ur50_lidar.xacro" />
+  <xacro:include filename="$(find magni_description)/urdf/sensors/light_sensor.xacro" />
   <!-- Robot base_link -->
   <link name="base_link">
@@ -232,3 +233,8 @@
     </joint>
   </xacro:if>
+  <!-- Define light sensor -->
+  <xacro:light_sensor name="light_sensor" connected_to="base_link">
+    <origin xyz="0.37 0 0"
+      rpy="0 0 0"/>
+  </xacro:light_sensor>
 </robot>

Commit message: Fix urdf meshes

File: magni_description/urdf/magni.urdf.xacro (robot description, xacro)
@@ -24,5 +24,5 @@
       <origin xyz="${-wheel_xpos} 0 ${-wheel_r+0.071}" rpy="0 0 0" />
       <geometry>
-        <mesh filename="package://magni_description/meshes/magni_body.dae" />
+        <mesh filename="$(find magni_description)/meshes/magni_body.dae" />
       </geometry>
     </visual>
@@ -30,5 +30,5 @@
       <origin xyz="${-wheel_xpos-0.169} 0.17 ${-wheel_r+0.09}" rpy="0 0 ${pi}" />
       <geometry>
-        <mesh filename="package://magni_description/meshes/caster_wheel.dae" />
+        <mesh filename="$(find magni_description)/meshes/caster_wheel.dae" />
       </geometry>
     </visual>
@@ -36,5 +36,5 @@
       <origin xyz="${-wheel_xpos-0.169} -0.17 ${-wheel_r+0.09}" rpy="0 0 ${pi}" />
       <geometry>
-        <mesh filename="package://magni_description/meshes/caster_wheel.dae" />
+        <mesh filename="$(find magni_description)/meshes/caster_wheel.dae" />
       </geometry>
     </visual>
@@ -71,5 +71,5 @@
         <origin xyz="0 0 0.005" rpy="0 0 0" />
         <geometry>
-          <mesh filename="package://magni_description/meshes/magni_tower.dae" />
+          <mesh filename="$(find magni_description)/meshes/magni_tower.dae" />
         </geometry>
       </visual>
@@ -115,5 +115,5 @@
         <origin xyz="0 0 0.005" rpy="0 0 0" />
         <geometry>
-          <mesh filename="package://magni_description/meshes/magni_shell.dae" />
+          <mesh filename="$(find magni_description)/meshes/magni_shell.dae" />
         </geometry>
       </visual>
