Commit message: package changes

File: magni_description/urdf/magni.urdf.xacro (robot description, xacro)
@@ -140,5 +140,5 @@
         <origin xyz="${-0.071*reflect} 0 0" rpy="0 ${(reflect-1)*pi/2} 0" />
         <geometry>
-          <mesh filename="package://magni_description/meshes/front_wheel.dae" />
+          <mesh filename="$(find magni_description)/meshes/front_wheel.dae" />
         </geometry>
       </visual>

File: magni_description/urdf/sensors/raspi_camera.xacro (robot description, xacro)
@@ -13,5 +13,5 @@
         <origin xyz="0 0 0" rpy="0 0 ${-pi/2}" />
         <geometry>
-          <mesh filename="package://magni_description/meshes/sensors/raspi_camera.dae" />
+          <mesh filename="$(find magni_description)/meshes/sensors/raspi_camera.dae" />
         </geometry>
       </visual>

File: magni_description/urdf/sensors/sonar_hc-sr04.xacro (robot description, xacro)
@@ -13,5 +13,5 @@
         <origin xyz="-0.006 0 0" rpy="${pi/2} 0 ${pi/2}" />
         <geometry>
-          <mesh filename="package://magni_description/meshes/sensors/sonar_hc-sr04.dae" />
+          <mesh filename="$(find magni_description)/meshes/sensors/sonar_hc-sr04.dae" />
         </geometry>
       </visual>

File: magni_description/urdf/sensors/ur50_lidar.xacro (robot description, xacro)
@@ -13,5 +13,5 @@
       <origin xyz="0 0 -0.03" rpy="0 0 0" />
       <geometry>
-        <mesh filename="package://magni_description/meshes/sensors/ur50_lidar.dae" />
+        <mesh filename="$(find magni_description)/meshes/sensors/ur50_lidar.dae" />
       </geometry>
     </visual>

File: magni_description/urdf/sensors/ur_c1_lidar.xacro (robot description, xacro)
@@ -13,5 +13,5 @@
       <origin xyz="0 0 -0.03" rpy="0 0 0" />
       <geometry>
-        <mesh filename="package://magni_description/meshes/sensors/ur_c1_lidar.dae" />
+        <mesh filename="$(find magni_description)/meshes/sensors/ur_c1_lidar.dae" />
       </geometry>
     </visual>

File: magni_description/urdf/tower/tower.urdf.xacro (robot description, xacro)
@@ -24,5 +24,5 @@
       <origin xyz="${-wheel_xpos} 0 ${-wheel_r+0.071}" rpy="0 0 0" />
       <geometry>
-        <mesh filename="package://magni_description/meshes/magni_body.dae" />
+        <mesh filename="$(find magni_description)/meshes/magni_body.dae" />
       </geometry>
     </visual>
@@ -30,5 +30,5 @@
       <origin xyz="${-wheel_xpos-0.169} 0.17 ${-wheel_r+0.09}" rpy="0 0 ${pi}" />
       <geometry>
-        <mesh filename="package://magni_description/meshes/caster_wheel.dae" />
+        <mesh filename="$(find magni_description)/meshes/caster_wheel.dae" />
       </geometry>
     </visual>
@@ -36,5 +36,5 @@
       <origin xyz="${-wheel_xpos-0.169} -0.17 ${-wheel_r+0.09}" rpy="0 0 ${pi}" />
       <geometry>
-        <mesh filename="package://magni_description/meshes/caster_wheel.dae" />
+        <mesh filename="$(find magni_description)/meshes/caster_wheel.dae" />
       </geometry>
     </visual>
@@ -71,5 +71,5 @@
         <origin xyz="0 0 0.005" rpy="0 0 0" />
         <geometry>
-          <mesh filename="package://magni_description/meshes/magni_tower.dae" />
+          <mesh filename="$(find magni_description)/meshes/magni_tower.dae" />
         </geometry>
       </visual>
@@ -115,5 +115,5 @@
         <origin xyz="0 0 0.005" rpy="0 0 0" />
         <geometry>
-          <mesh filename="package://magni_description/meshes/magni_shell.dae" />
+          <mesh filename="$(find magni_description)/meshes/magni_shell.dae" />
         </geometry>
       </visual>
@@ -140,5 +140,5 @@
         <origin xyz="${-0.071*reflect} 0 0" rpy="0 ${(reflect-1)*pi/2} 0" />
         <geometry>
-          <mesh filename="package://magni_description/meshes/front_wheel.dae" />
+          <mesh filename="$(find magni_description)/meshes/front_wheel.dae" />
         </geometry>
       </visual>

Commit message: lidar fix ur_c1_lidar

File: magni_description/urdf/magni.urdf.xacro (robot description, xacro)
@@ -212,7 +212,11 @@
   </xacro:if>
   <!-- Define Lidar -->
+<!-- hardcoded values for the lidar extrinsics -->
+  <xacro:property name="lidar_extrinsics_file" value="$(find magni_description)/urdf/extrinsics/lidar_extrinsics_top_plate_center.yaml"/>
   <xacro:if value="${lidar_extrinsics_file != ''}">
+  <!-- <xacro:if value="${lidar_extrinsics_file}"> -->
     <xacro:property name="lidar_extrinsics" value="${xacro.load_yaml(lidar_extrinsics_file)}"/>
-    <xacro:ur_c1_lidar name="laser" connected_to="base_link">
+    <!-- <xacro:ur_c1_lidar name="laser" connected_to="base_link"> -->
+    <xacro:ur_c1_lidar name="ur_c1_lidar" connected_to="base_link">
       <origin xyz="${lidar_extrinsics['x']} ${lidar_extrinsics['y']} ${lidar_extrinsics['z']}"
         rpy="${lidar_extrinsics['roll']} ${lidar_extrinsics['pitch']} ${lidar_extrinsics['yaw']}"/>

File: magni_description/urdf/sensors/sonar_hc-sr04.xacro (robot description, xacro)
@@ -51,5 +51,5 @@
         </ray>
         <!-- Gazebo-ROS interface plugin -->
-        <plugin filename="libgazebo_ros_range.so" name="gazebo_ros_range">
+        <!-- <plugin filename="libgazebo_ros_range.so" name="gazebo_ros_range">
           <gaussianNoise>0.015</gaussianNoise>
           <alwaysOn>true</alwaysOn>
@@ -59,5 +59,5 @@
           <fov>0.5</fov>
           <radiation>ultrasound</radiation>
-        </plugin>
+        </plugin> -->
       </sensor>
     </gazebo>

File: magni_description/urdf/sensors/ur_c1_lidar.xacro (robot description, xacro)
@@ -30,5 +30,6 @@
       <visualize>false</visualize>
       <update_rate>20</update_rate>
-      <ray>
+      <!-- <ray> -->
+      <lidar>
         <scan>
           <horizontal>
@@ -53,8 +54,10 @@
           <stddev>0.01</stddev>
         </noise>
-      </ray>
+      <!-- </ray> -->
+      </lidar>
       <!--<plugin name="gazebo_ros_head_hokuyo_controller" filename="libgazebo_ros_gpu_laser.so">-->
       <!-- <plugin name="gazebo_ros_head_hokuyo_controller" filename="libgazebo_ros_laser.so"> -->
-        <topicName>/scan</topicName>
+        <!-- <topicName>/scan</topicName> -->
+        <topic>/scan</topic>
         <!-- <frameName>${name}</frameName> -->
         <gz_frame_id>${name}</gz_frame_id>

Commit message: odom frame added

File: magni_description/urdf/magni.urdf.xacro (robot description, xacro)
@@ -241,3 +241,10 @@
     </joint>
   </ros2_control>
+  <!-- Odometry Frame -->
+<link name="odom"/>
+<joint name="odom_joint" type="fixed">
+  <parent link="odom"/>
+  <child link="base_footprint"/>
+  <origin xyz="0 0 0" rpy="0 0 0"/>
+</joint>
 </robot>

Commit message: added odom to launch from urdf

File: magni_description/urdf/magni.urdf.xacro (robot description, xacro)
@@ -242,9 +242,15 @@
   </ros2_control>
   <!-- Odometry Frame -->
-<link name="odom"/>
+<!-- <link name="odom"/> -->
+<!-- <joint name="odom_joint" type="fixed"> -->
+<!-- <joint name="odom_joint" type="floating"> -->
+  <!-- <parent link="odom"/>
+  <child link="base_footprint"/>
+  <origin xyz="0 0 0" rpy="0 0 0"/>
+</joint> -->
+<!-- <link name="odom"/>
 <joint name="odom_joint" type="fixed">
   <parent link="odom"/>
-  <child link="base_footprint"/>
-  <origin xyz="0 0 0" rpy="0 0 0"/>
-</joint>
+  <child link="base_link"/>
+</joint> -->
 </robot>

Commit message: added ddom to urdf

File: magni_description/urdf/magni.urdf.xacro (robot description, xacro)
@@ -242,11 +242,11 @@
   </ros2_control>
   <!-- Odometry Frame -->
-<!-- <link name="odom"/> -->
+<link name="odom"/>
 <!-- <joint name="odom_joint" type="fixed"> -->
-<!-- <joint name="odom_joint" type="floating"> -->
-  <!-- <parent link="odom"/>
+<joint name="odom_joint" type="floating">
+  <parent link="odom"/>
   <child link="base_footprint"/>
   <origin xyz="0 0 0" rpy="0 0 0"/>
-</joint> -->
+</joint>
 <!-- <link name="odom"/>
 <joint name="odom_joint" type="fixed">

Commit message: changes to the launchfile and controller manager parameters

File: magni_description/urdf/magni.urdf.xacro (robot description, xacro)
@@ -241,16 +241,3 @@
     </joint>
   </ros2_control>
-  <!-- Odometry Frame -->
-<link name="odom"/>
-<!-- <joint name="odom_joint" type="fixed"> -->
-<joint name="odom_joint" type="floating">
-  <parent link="odom"/>
-  <child link="base_footprint"/>
-  <origin xyz="0 0 0" rpy="0 0 0"/>
-</joint>
-<!-- <link name="odom"/>
-<joint name="odom_joint" type="fixed">
-  <parent link="odom"/>
-  <child link="base_link"/>
-</joint> -->
 </robot>

Commit message: deep study of refacotring, adding gnss extrinsics...

File: magni_description/urdf/magni.urdf.xacro (robot description, xacro)
@@ -11,4 +11,6 @@
   <xacro:arg name="lidar_extrinsics_file" default=""/>
   <xacro:property name="lidar_extrinsics_file" value="$(arg lidar_extrinsics_file)"/>
+  <xacro:arg name="gps_extrinsics_file" default=""/>
+  <xacro:property name="gps_extrinsics_file" value="$(arg gps_extrinsics_file)"/>
   <xacro:property name="wheel_r" value="0.1" />
   <xacro:property name="wheel_xpos" value="0.11" />
@@ -223,4 +225,44 @@
     </xacro:ur_c1_lidar>
   </xacro:if>
+  <xacro:if value="${gps_extrinsics_file != ''}">
+      <xacro:property name="gps_extrinsics" value="${xacro.load_yaml(gps_extrinsics_file)}"/>
+      <link name="gps_link">
+        <visual>
+          <geometry>
+            <box size="0.05 0.05 0.02"/>
+          </geometry>
+          <material name="black"/>
+        </visual>
+      </link>
+      <joint name="gps_joint" type="fixed">
+        <parent link="base_link"/>
+        <child link="gps_link"/>
+        <origin xyz="${gps_extrinsics['x']} ${gps_extrinsics['y']} ${gps_extrinsics['z']}"
+          rpy="${gps_extrinsics['roll']} ${gps_extrinsics['pitch']} ${gps_extrinsics['yaw']}"/>
+      </joint>
+      <gazebo reference="gps_link">
+        <sensor name="navsat" type="navsat">
+          <always_on>1</always_on>
+          <update_rate>1</update_rate>
+          <topic>navsat</topic>
+          <navsat>
+            <position_sensing>
+              <horizontal>
+                <noise type="gaussian">
+                  <mean>0.0</mean>
+                  <stddev>0.01</stddev>
+                </noise>
+              </horizontal>
+              <vertical>
+                <noise type="gaussian">
+                  <mean>0.0</mean>
+                  <stddev>0.01</stddev>
+                </noise>
+              </vertical>
+            </position_sensing>
+          </navsat>
+        </sensor>
+      </gazebo>
+    </xacro:if>
  <!-- ROS 2 Control block -->
   <ros2_control name="ubiquity_motor_ros2/MotorHardware" type="system">
