Commit message: Removed duplicate launch of diff drive controlller..

File: magni_description/urdf/magni.transmission.xacro (robot description, xacro)
@@ -1,24 +1,4 @@
 <?xml version="1.0"?>
 <robot xmlns:xacro="http://wiki.ros.org/xacro">
-  <ros2_control name="GazeboSystem" type="system">
-    <hardware>
-      <plugin>gz_ros2_control/GazeboSimSystem</plugin>
-    </hardware>
-    <joint name="left_wheel_joint">
-      <command_interface name="velocity">
-        <param name="min">-10</param>
-        <param name="max">10</param>
-      </command_interface>
-      <state_interface name="position"/>
-      <state_interface name="velocity"/>
-    </joint>
-    <joint name="right_wheel_joint">
-      <command_interface name="velocity">
-        <param name="min">-10</param>
-        <param name="max">10</param>
-      </command_interface>
-      <state_interface name="position"/>
-      <state_interface name="velocity"/>
-    </joint>
-  </ros2_control>
+  <!-- Intentionally empty: ros2_control is defined in each robot URDF to avoid duplicate controller_managers. -->
 </robot>

File: magni_description/urdf/magni_base.urdf.xacro (robot description, xacro)
@@ -136,10 +136,3 @@
     </joint>
   </ros2_control>
-  <xacro:if value="$(arg use_sim)">
-    <gazebo>
-        <plugin filename="gz_ros2_control-system" name="gz_ros2_control::GazeboSimROS2ControlPlugin">
-            <parameters>$(find magni_gazebo)/config/diff_drive_controller.yaml</parameters>
-        </plugin>
-    </gazebo>
-  </xacro:if>
 </robot>

File: magni_description/urdf/robots/gen_6_microtractor.urdf.xacro (robot description, xacro)
@@ -142,11 +142,4 @@
     </joint>
   </ros2_control>
-  <xacro:if value="$(arg use_sim)">
-    <gazebo>
-        <plugin filename="gz_ros2_control-system" name="gz_ros2_control::GazeboSimROS2ControlPlugin">
-            <parameters>$(find magni_gazebo)/config/diff_drive_controller.yaml</parameters>
-        </plugin>
-    </gazebo>
-  </xacro:if>
   <!-- Lidar (High Lidar) -->
   <xacro:ur50_lidar name="laser" connected_to="base_link">

File: magni_description/urdf/robots/gen_6_midi.urdf.xacro (robot description, xacro)
@@ -141,11 +141,4 @@
     </joint>
   </ros2_control>
-  <xacro:if value="$(arg use_sim)">
-    <gazebo>
-        <plugin filename="gz_ros2_control-system" name="gz_ros2_control::GazeboSimROS2ControlPlugin">
-            <parameters>$(find magni_gazebo)/config/diff_drive_controller.yaml</parameters>
-        </plugin>
-    </gazebo>
-  </xacro:if>
   <!-- Lidar Configuration for Midi (Top Plate) -->
   <xacro:ur_c1_lidar name="laser" connected_to="base_link">

File: magni_description/urdf/robots/gen_6_mini.urdf.xacro (robot description, xacro)
@@ -140,11 +140,4 @@
     </joint>
   </ros2_control>
-  <xacro:if value="$(arg use_sim)">
-    <gazebo>
-        <plugin filename="gz_ros2_control-system" name="gz_ros2_control::GazeboSimROS2ControlPlugin">
-            <parameters>$(find magni_gazebo)/config/diff_drive_controller.yaml</parameters>
-        </plugin>
-    </gazebo>
-  </xacro:if>
   <!-- Lidar Configuration for Mini (Top Plate) -->
   <xacro:ur_c1_lidar name="laser" connected_to="base_link">
