Commit message: Revert "Jazzy devel gz sim test"

File: magni_description/urdf/magni.gazebo.xacro (robot description, xacro)
@@ -1,5 +1,5 @@
 <?xml version="1.0"?>
 <robot xmlns:xacro="http://wiki.ros.org/xacro">
-    <!-- <gazebo>
+    <gazebo>
         <plugin name="gazebo_ros_control" filename="libgazebo_ros_control.so">
             <legacyModeNS>true</legacyModeNS>
@@ -12,21 +12,4 @@
             <topicName>exact_pose</topicName>
             <frameName>map</frameName>
-        </plugin>
-    </gazebo> -->
-    <gazebo>
-        <plugin filename="gz-sim-diff-drive-system" name="gz::sim::systems::DiffDrive">
-            <right_joint>right_wheel_joint</right_joint>
-            <left_joint>left_wheel_joint</left_joint>
-            <!-- <wheel_separation>${wheel_separation}</wheel_separation> -->
-            <!-- <wheel_radius>${wheel_radius}</wheel_radius> -->
-            <!-- <max_linear_acceleration>${max_linear_acceleration}</max_linear_acceleration> -->
-            <odom_publish_frequency>100</odom_publish_frequency>
-            <topic>cmd_vel</topic>
-            <odom_topic>odom</odom_topic>
-        </plugin>
-        <plugin filename="gz-sim-joint-state-publisher-system" name="gz::sim::systems::JointStatePublisher">
-            <topic>joint_states</topic>
-            <joint_name>right_wheel_joint</joint_name>
-            <joint_name>left_wheel_joint</joint_name>
         </plugin>
     </gazebo>

File: magni_description/urdf/magni.urdf.xacro (robot description, xacro)
@@ -18,5 +18,5 @@
   <xacro:include filename="$(find magni_description)/urdf/sensors/sonar_hc-sr04.xacro" />
   <xacro:include filename="$(find magni_description)/urdf/sensors/raspi_camera.xacro" />
-  <xacro:include filename="$(find magni_description)/urdf/sensors/ur_c1_lidar.xacro" />
+  <xacro:include filename="$(find magni_description)/urdf/sensors/ur50_lidar.xacro" />
   <!-- Robot base_link -->
   <link name="base_link">
@@ -24,5 +24,5 @@
       <origin xyz="${-wheel_xpos} 0 ${-wheel_r+0.071}" rpy="0 0 0" />
       <geometry>
-        <mesh filename="$(find magni_description)/meshes/magni_body.dae" />
+        <mesh filename="package://magni_description/meshes/magni_body.dae" />
       </geometry>
     </visual>
@@ -30,5 +30,5 @@
       <origin xyz="${-wheel_xpos-0.169} 0.17 ${-wheel_r+0.09}" rpy="0 0 ${pi}" />
       <geometry>
-        <mesh filename="$(find magni_description)/meshes/caster_wheel.dae" />
+        <mesh filename="package://magni_description/meshes/caster_wheel.dae" />
       </geometry>
     </visual>
@@ -36,5 +36,5 @@
       <origin xyz="${-wheel_xpos-0.169} -0.17 ${-wheel_r+0.09}" rpy="0 0 ${pi}" />
       <geometry>
-        <mesh filename="$(find magni_description)/meshes/caster_wheel.dae" />
+        <mesh filename="package://magni_description/meshes/caster_wheel.dae" />
       </geometry>
     </visual>
@@ -71,5 +71,5 @@
         <origin xyz="0 0 0.005" rpy="0 0 0" />
         <geometry>
-          <mesh filename="$(find magni_description)/meshes/magni_tower.dae" />
+          <mesh filename="package://magni_description/meshes/magni_tower.dae" />
         </geometry>
       </visual>
@@ -115,5 +115,5 @@
         <origin xyz="0 0 0.005" rpy="0 0 0" />
         <geometry>
-          <mesh filename="$(find magni_description)/meshes/magni_shell.dae" />
+          <mesh filename="package://magni_description/meshes/magni_shell.dae" />
         </geometry>
       </visual>
@@ -140,5 +140,5 @@
         <origin xyz="${-0.071*reflect} 0 0" rpy="0 ${(reflect-1)*pi/2} 0" />
         <geometry>
-          <mesh filename="$(find magni_description)/meshes/front_wheel.dae" />
+          <mesh filename="package://magni_description/meshes/front_wheel.dae" />
         </geometry>
       </visual>
@@ -214,8 +214,8 @@
   <xacro:if value="${lidar_extrinsics_file != ''}">
     <xacro:property name="lidar_extrinsics" value="${xacro.load_yaml(lidar_extrinsics_file)}"/>
-    <xacro:ur_c1_lidar name="laser" connected_to="base_link">
+    <xacro:ur50_lidar name="laser" connected_to="base_link">
       <origin xyz="${lidar_extrinsics['x']} ${lidar_extrinsics['y']} ${lidar_extrinsics['z']}"
         rpy="${lidar_extrinsics['roll']} ${lidar_extrinsics['pitch']} ${lidar_extrinsics['yaw']}"/>
-    </xacro:ur_c1_lidar>
+    </xacro:ur50_lidar>
   </xacro:if>
  <!-- ROS 2 Control block -->

File: magni_description/urdf/sensors/raspi_camera.xacro (robot description, xacro)
@@ -13,5 +13,5 @@
         <origin xyz="0 0 0" rpy="0 0 ${-pi/2}" />
         <geometry>
-          <mesh filename="$(find magni_description)/meshes/sensors/raspi_camera.dae" />
+          <mesh filename="package://magni_description/meshes/sensors/raspi_camera.dae" />
         </geometry>
       </visual>

File: magni_description/urdf/sensors/sonar_hc-sr04.xacro (robot description, xacro)
@@ -13,5 +13,5 @@
         <origin xyz="-0.006 0 0" rpy="${pi/2} 0 ${pi/2}" />
         <geometry>
-          <mesh filename="$(find magni_description)/meshes/sensors/sonar_hc-sr04.dae" />
+          <mesh filename="package://magni_description/meshes/sensors/sonar_hc-sr04.dae" />
         </geometry>
       </visual>

File: magni_description/urdf/sensors/ur50_lidar.xacro (robot description, xacro)
@@ -13,5 +13,5 @@
       <origin xyz="0 0 -0.03" rpy="0 0 0" />
       <geometry>
-        <mesh filename="$(find magni_description)/meshes/sensors/ur50_lidar.dae" />
+        <mesh filename="package://magni_description/meshes/sensors/ur50_lidar.dae" />
       </geometry>
     </visual>
@@ -25,6 +25,5 @@
   <gazebo reference="${name}">
     <!--<sensor type="gpu_ray" name="${name}_sensor>-->
-    <!-- <sensor type="ray" name="${name}_sensor"> -->
-    <sensor type="gpu_lidar" name="${name}_sensor">
+    <sensor type="ray" name="${name}_sensor">
       <pose>0 0 0 0 0 0</pose>
       <visualize>false</visualize>
@@ -55,8 +54,7 @@
       </ray>
       <!--<plugin name="gazebo_ros_head_hokuyo_controller" filename="libgazebo_ros_gpu_laser.so">-->
-      <!-- <plugin name="gazebo_ros_head_hokuyo_controller" filename="libgazebo_ros_laser.so"> -->
+      <plugin name="gazebo_ros_head_hokuyo_controller" filename="libgazebo_ros_laser.so">
         <topicName>/scan</topicName>
-        <!-- <frameName>${name}</frameName> -->
-        <gz_frame_id>${name}</gz_frame_id>
+        <frameName>${name}</frameName>
       </plugin>
     </sensor>

File: magni_description/urdf/tower/sensors/ur50_lidar.xacro (robot description, xacro)
@@ -13,5 +13,5 @@
       <origin xyz="0 0 -0.03" rpy="0 0 0" />
       <geometry>
-        <mesh filename="$(find magni_description)/meshes/sensors/ur50_lidar.dae" />
+        <mesh filename="package://magni_description/meshes/sensors/ur50_lidar.dae" />
       </geometry>
     </visual>

File: magni_description/urdf/tower/tower.urdf.xacro (robot description, xacro)
@@ -24,5 +24,5 @@
       <origin xyz="${-wheel_xpos} 0 ${-wheel_r+0.071}" rpy="0 0 0" />
       <geometry>
-        <mesh filename="$(find magni_description)/meshes/magni_body.dae" />
+        <mesh filename="package://magni_description/meshes/magni_body.dae" />
       </geometry>
     </visual>
@@ -30,5 +30,5 @@
       <origin xyz="${-wheel_xpos-0.169} 0.17 ${-wheel_r+0.09}" rpy="0 0 ${pi}" />
       <geometry>
-        <mesh filename="$(find magni_description)/meshes/caster_wheel.dae" />
+        <mesh filename="package://magni_description/meshes/caster_wheel.dae" />
       </geometry>
     </visual>
@@ -36,5 +36,5 @@
       <origin xyz="${-wheel_xpos-0.169} -0.17 ${-wheel_r+0.09}" rpy="0 0 ${pi}" />
       <geometry>
-        <mesh filename="$(find magni_description)/meshes/caster_wheel.dae" />
+        <mesh filename="package://magni_description/meshes/caster_wheel.dae" />
       </geometry>
     </visual>
@@ -71,5 +71,5 @@
         <origin xyz="0 0 0.005" rpy="0 0 0" />
         <geometry>
-          <mesh filename="$(find magni_description)/meshes/magni_tower.dae" />
+          <mesh filename="package://magni_description/meshes/magni_tower.dae" />
         </geometry>
       </visual>
@@ -115,5 +115,5 @@
         <origin xyz="0 0 0.005" rpy="0 0 0" />
         <geometry>
-          <mesh filename="$(find magni_description)/meshes/magni_shell.dae" />
+          <mesh filename="package://magni_description/meshes/magni_shell.dae" />
         </geometry>
       </visual>
@@ -140,5 +140,5 @@
         <origin xyz="${-0.071*reflect} 0 0" rpy="0 ${(reflect-1)*pi/2} 0" />
         <geometry>
-          <mesh filename="$(find magni_description)/meshes/front_wheel.dae" />
+          <mesh filename="package://magni_description/meshes/front_wheel.dae" />
         </geometry>
       </visual>

Commit message: teleop keyboard functionality added

File: magni_description/urdf/magni.gazebo.xacro (robot description, xacro)
@@ -1,4 +1,8 @@
 <?xml version="1.0"?>
 <robot xmlns:xacro="http://wiki.ros.org/xacro">
+<xacro:property name="wheel_r" value="0.1" />
+<xacro:property name="chassis_width" value="0.268"/>
+<xacro:property name="wheel_thickness" value="0.05" />
+<xacro:property name="wheel_separation" value="${chassis_width + wheel_thickness}"/>
     <!-- <gazebo>
         <plugin name="gazebo_ros_control" filename="libgazebo_ros_control.so">
@@ -18,6 +22,6 @@
             <right_joint>right_wheel_joint</right_joint>
             <left_joint>left_wheel_joint</left_joint>
-            <!-- <wheel_separation>${wheel_separation}</wheel_separation> -->
-            <!-- <wheel_radius>${wheel_radius}</wheel_radius> -->
+            <wheel_separation>${wheel_separation}</wheel_separation>
+            <wheel_radius>${wheel_r}</wheel_radius>
             <!-- <max_linear_acceleration>${max_linear_acceleration}</max_linear_acceleration> -->
             <odom_publish_frequency>100</odom_publish_frequency>

Commit message: fix(sim): migrate to gz_ros2_control for ROS 2 Jazzy
- Replace legacy libgazebo_ros_control.so with libgz_ros2_control-system.so in magni.gazebo.xacro.
- Rewrite magni.transmission.xacro to use <ros2_control> tag instead of legacy <transmission>.
- Disable direct cmd_vel bridging in gz_bridge.yaml to prevent conflicts with ros2_control.

File: magni_description/urdf/magni.gazebo.xacro (robot description, xacro)
@@ -2,6 +2,6 @@
 <robot xmlns:xacro="http://wiki.ros.org/xacro">
     <gazebo>
-        <plugin name="gazebo_ros_control" filename="libgazebo_ros_control.so">
-            <legacyModeNS>true</legacyModeNS>
+        <plugin filename="libgz_ros2_control-system.so" name="gz_ros2_control::GazeboSimROS2ControlPlugin">
+            <parameters>$(find magni_gazebo)/config/diff_drive_controller.yaml</parameters>
         </plugin>
     </gazebo>

File: magni_description/urdf/magni.transmission.xacro (robot description, xacro)
@@ -1,23 +1,24 @@
 <?xml version="1.0"?>
 <robot xmlns:xacro="http://wiki.ros.org/xacro">
-    <transmission name="left_wheel_transmission">
-        <type>transmission_interface/SimpleTransmission</type>
-        <joint name="left_wheel_joint">
-            <hardwareInterface>hardware_interface/VelocityJointInterface</hardwareInterface>
-        </joint>
-        <actuator name="left_wheel_actuator">
-            <mechanicalReduction>1</mechanicalReduction>
-            <hardwareInterface>VelocityJointInterface</hardwareInterface>
-        </actuator>
-    </transmission>
-    <transmission name="right_wheel_transmission">
-        <type>transmission_interface/SimpleTransmission</type>
-        <joint name="right_wheel_joint">
-            <hardwareInterface>hardware_interface/VelocityJointInterface</hardwareInterface>
-        </joint>
-        <actuator name="right_wheel_actuator">
-            <mechanicalReduction>1</mechanicalReduction>
-            <hardwareInterface>VelocityJointInterface</hardwareInterface>
-        </actuator>
-    </transmission>
+  <ros2_control name="GazeboSystem" type="system">
+    <hardware>
+      <plugin>gz_ros2_control/GazeboSimSystem</plugin>
+    </hardware>
+    <joint name="left_wheel_joint">
+      <command_interface name="velocity">
+        <param name="min">-10</param>
+        <param name="max">10</param>
+      </command_interface>
+      <state_interface name="position"/>
+      <state_interface name="velocity"/>
+    </joint>
+    <joint name="right_wheel_joint">
+      <command_interface name="velocity">
+        <param name="min">-10</param>
+        <param name="max">10</param>
+      </command_interface>
+      <state_interface name="position"/>
+      <state_interface name="velocity"/>
+    </joint>
+  </ros2_control>
 </robot>
