Commit message: Paper background added to markers

File: magni_gazebo/urdf/fiducials/aruco_marker.xacro (robot description, xacro)
@@ -15,5 +15,5 @@
             <visual>
                 <geometry>
-                    <box size="0.14 0.14 0.001"/>
+                    <box size="0.14 0.14 0.003"/>
                 </geometry>
             </visual>
@@ -23,4 +23,18 @@
             <turnGravityOff>true</turnGravityOff>
         </gazebo>
+        <joint name="${prefix}${marker_id}paper_joint" type="fixed">
+            <parent link="${prefix}${marker_id}base_link"/>
+            <child link="${prefix}${marker_id}paper_link"/>
+        </joint>
+        <link name="${prefix}${marker_id}paper_link">
+            <visual>
+                <geometry>
+                    <box size="0.297 0.21 0.001"/>
+                </geometry>
+            </visual>
+        </link>
+        <gazebo reference="${prefix}${marker_id}paper_link">
+            <material>MagniWorld/White</material>
+        </gazebo>
     </xacro:macro>
 </robot>
