Commit message: Fix fiducial rotation

File: magni_gazebo/urdf/fiducials/fiducial_grid_ground.urdf.xacro (robot description, xacro)
@@ -8,23 +8,23 @@
     <link name="world"/>
     <xacro:aruco_marker prefix="$(arg prefix)" marker_id="0" parent="world">
-        <origin xyz="${1*grid_size} 0 ${height}" rpy="${pi} 0 0"/>
+        <origin xyz="${1*grid_size} 0 ${height}" rpy="0 0 0"/>
     </xacro:aruco_marker>
     <xacro:aruco_marker prefix="$(arg prefix)" marker_id="1" parent="world">
-        <origin xyz="${2*grid_size} 0 ${height}" rpy="${pi} 0 0"/>
+        <origin xyz="${2*grid_size} 0 ${height}" rpy="0 0 0"/>
     </xacro:aruco_marker>
     <xacro:aruco_marker prefix="$(arg prefix)" marker_id="2" parent="world">
-        <origin xyz="${3*grid_size} 0 ${height}" rpy="${pi} 0 0"/>
+        <origin xyz="${3*grid_size} 0 ${height}" rpy="0 0 0"/>
     </xacro:aruco_marker>
     <xacro:aruco_marker prefix="$(arg prefix)" marker_id="3" parent="world">
-        <origin xyz="${4*grid_size} 0 ${height}" rpy="${pi} 0 0"/>
+        <origin xyz="${4*grid_size} 0 ${height}" rpy="0 0 0"/>
     </xacro:aruco_marker>
     <xacro:aruco_marker prefix="$(arg prefix)" marker_id="4" parent="world">
-        <origin xyz="${5*grid_size} 0 ${height}" rpy="${pi} 0 0"/>
+        <origin xyz="${5*grid_size} 0 ${height}" rpy="0 0 0"/>
     </xacro:aruco_marker>
     <xacro:aruco_marker prefix="$(arg prefix)" marker_id="5" parent="world">
-        <origin xyz="${6*grid_size} 0 ${height}" rpy="${pi} 0 0"/>
+        <origin xyz="${6*grid_size} 0 ${height}" rpy="0 0 0"/>
     </xacro:aruco_marker>
     <xacro:aruco_marker prefix="$(arg prefix)" marker_id="6" parent="world">
-        <origin xyz="${7*grid_size} 0 ${height}" rpy="${pi} 0 0"/>
+        <origin xyz="${7*grid_size} 0 ${height}" rpy="0 0 0"/>
     </xacro:aruco_marker>
 </robot>
