Commit message: Implemented quickfiy suggestion in #140

File: magni_description/urdf/sensors/raspi_camera.xacro (robot description, xacro)
@@ -28,5 +28,5 @@
       <parent link="${name}"/>
       <child link="${name}_sensor"/>
-      <origin xyz="0 0 0.012" rpy="${pi/2} ${-pi/2} 0" />
+      <origin xyz="0 0 0.012" rpy="${-pi/2} 0 ${-pi/2}" />
     </joint>
     <!-- Gazebo sensor plugin -->

Commit message: Minor camera URDF refactoring.
To prevent confusing with additional link for Gazebo camera sensor.

File: magni_description/urdf/sensors/raspi_camera.xacro (robot description, xacro)
@@ -23,13 +23,13 @@
       </collision>
     </link>
-    <!-- Additional link for camera sensor to orient camera direction -->
-    <link name="${name}_sensor"/>
-    <joint name="${name}_sensor_joint" type="fixed">
+    <!-- Additional link for camera Gazebo sensor to orient camera direction (it is used only for Gazebo simulation) -->
+    <link name="${name}_gazebo_sensor"/>
+    <joint name="${name}_gazebo_sensor_joint" type="fixed">
       <parent link="${name}"/>
-      <child link="${name}_sensor"/>
+      <child link="${name}_gazebo_sensor"/>
       <origin xyz="0 0 0.012" rpy="${pi/2} ${-pi/2} 0" />
     </joint>
     <!-- Gazebo sensor plugin -->
-    <gazebo reference="${name}_sensor">
+    <gazebo reference="${name}_gazebo_sensor">
       <sensor type="camera" name="camera1">
         <visualize>false</visualize>
