Commit message: disabling collision for sonars, solving #200

File: magni_description/urdf/sensors/sonar_hc-sr04.xacro (robot description, xacro)
@@ -16,10 +16,11 @@
         </geometry>
       </visual>
-      <collision>
+      <!-- removing colisions from sonars solves issue https://github.com/UbiquityRobotics/magni_robot/issues/200 -->
+      <!-- <collision>
         <origin xyz="0 0 0" rpy="0 0 0" />
         <geometry>
           <box size="0.02 0.044 0.021"/>
         </geometry>
-      </collision>
+      </collision> -->
     </link>
     <!-- Gazebo sensor plugin -->
