Commit message: Corrected the ur50 gazebo sim specs

File: magni_description/urdf/sensors/ur50_lidar.xacro (robot description, xacro)
@@ -11,5 +11,5 @@
   <link name="${name}">
     <visual>
-      <origin xyz="0 0 0" rpy="0 0 0" />
+      <origin xyz="0 0 -0.03" rpy="0 0 0" />
       <geometry>
         <mesh filename="package://magni_description/meshes/sensors/ur50_lidar.dae" />
@@ -28,5 +28,5 @@
       <pose>0 0 0 0 0 0</pose>
       <visualize>false</visualize>
-      <update_rate>15</update_rate>
+      <update_rate>20</update_rate>
       <ray>
         <scan>
@@ -34,11 +34,11 @@
             <samples>811</samples>
             <!--<resolution>0.3333</resolution>-->
-            <min_angle>-2.3561925</min_angle>
-            <max_angle>2.3561925</max_angle>
+            <min_angle>-3.14</min_angle>
+            <max_angle>3.14</max_angle>
           </horizontal>
         </scan>
         <range>
-          <min>0.20</min>
-          <max>30.0</max>
+          <min>0.05</min>
+          <max>50.0</max>
           <resolution>0.01</resolution>
         </range>
