Commit message: typo change

File: magni_description/urdf/sensors/light_sensor.xacro (robot description, xacro)
@@ -1,5 +1,5 @@
 <?xml version="1.0" encoding="utf-8"?>
 <robot xmlns:xacro="http://wiki.ros.org/xacro">
-  <xacro:macro name="ligth_sensor" params="name:='' connected_to:='' *origin">
+  <xacro:macro name="light_sensor" params="name:='' connected_to:='' *origin">
   <xacro:unless value="${connected_to == ''}">
     <joint name="${name}_joint" type="fixed">

Commit message: Fix light sensor size and position in urdf

File: magni_description/urdf/sensors/light_sensor.xacro (robot description, xacro)
@@ -11,7 +11,7 @@
   <link name="${name}">
     <visual>
-      <origin xyz="0.37 0 0" rpy="0 0 0" />
+      <origin xyz="-0.255 0 0" rpy="1.57 0 1.57" />
       <geometry>
-        <mesh filename="package://magni_description/meshes/sensors/light_sensor.dae" />
+        <mesh filename="package://magni_description/meshes/sensors/light_sensor.dae"  scale="0.0012 0.0012 0.0012" />
       </geometry>
     </visual>
