Commit message: Implementing gnss sensor stream in gazebo

File: magni_description/urdf/robots/gen_6_microtractor.urdf.xacro (robot description, xacro)
@@ -184,6 +184,6 @@
   </xacro:raspi_camera>
   <!-- GPS (Top/Back) -->
-  <xacro:gps_antenna name="gps" parent="base_link">
-     <origin xyz="-0.10 0.0 0.25" rpy="0 0 0"/>
+  <xacro:gps_antenna name="gps" parent="base_link" simulate="true">
+     <origin xyz="-0.10 0.0 0.45" rpy="0 0 0"/>
   </xacro:gps_antenna>
   <!-- Lidar (Ubiquity Robotics C1) -->

File: magni_description/urdf/sensors/gps_antenna.xacro (robot description, xacro)
@@ -1,5 +1,5 @@
 <?xml version="1.0"?>
 <robot xmlns:xacro="http://wiki.ros.org/xacro">
-  <xacro:macro name="gps_antenna" params="name parent *origin">
+  <xacro:macro name="gps_antenna" params="name parent simulate:=false *origin">
     <joint name="${name}_joint" type="fixed">
       <xacro:insert_block name="origin" />
@@ -22,4 +22,79 @@
       </collision>
     </link>
+    <xacro:if value="${simulate}">
+      <gazebo reference="${name}_link">
+          <sensor name="${name}_sensor" type="navsat">
+              <always_on>1</always_on>
+              <update_rate>5.0</update_rate>
+              <topic>gnss/fix</topic>
+              <gz_frame_id>${name}_link</gz_frame_id>
+              <navsat>
+                  <position_sensing>
+                      <horizontal>
+                          <noise type="gaussian">
+                              <mean>0.0</mean>
+                              <stddev>0.1</stddev>
+                          </noise>
+                      </horizontal>
+                      <vertical>
+                          <noise type="gaussian">
+                              <mean>0.0</mean>
+                              <stddev>0.1</stddev>
+                          </noise>
+                      </vertical>
+                  </position_sensing>
+              </navsat>
+          </sensor>
+          <sensor name="${name}_imu" type="imu">
+              <always_on>1</always_on>
+              <update_rate>20.0</update_rate>
+              <topic>gnss/imu</topic>
+              <gz_frame_id>${name}_link</gz_frame_id>
+              <pose>0 0 0 0 0 3.14159265</pose>
+              <imu>
+                <angular_velocity>
+                  <x>
+                    <noise type="gaussian">
+                      <mean>0.0</mean>
+                      <stddev>2e-4</stddev>
+                    </noise>
+                  </x>
+                  <y>
+                    <noise type="gaussian">
+                      <mean>0.0</mean>
+                      <stddev>2e-4</stddev>
+                    </noise>
+                  </y>
+                  <z>
+                    <noise type="gaussian">
+                      <mean>0.0</mean>
+                      <stddev>2e-4</stddev>
+                    </noise>
+                  </z>
+                </angular_velocity>
+                <linear_acceleration>
+                  <x>
+                    <noise type="gaussian">
+                      <mean>0.0</mean>
+                      <stddev>1.7e-2</stddev>
+                    </noise>
+                  </x>
+                  <y>
+                    <noise type="gaussian">
+                      <mean>0.0</mean>
+                      <stddev>1.7e-2</stddev>
+                    </noise>
+                  </y>
+                  <z>
+                    <noise type="gaussian">
+                      <mean>0.0</mean>
+                      <stddev>1.7e-2</stddev>
+                    </noise>
+                  </z>
+                </linear_acceleration>
+              </imu>
+          </sensor>
+      </gazebo>
+    </xacro:if>
   </xacro:macro>
 </robot>
